File: Thermocouple-Data-Logger/Thermocouple Data Logger.sch (KiCad schematic (older format))
At the start: 16 parts

Commit message: Added a lot more to the schimatic
Parts:
- added C? (x2): 0.33uF, symbol device:C
- added D? (x2): D_Schottky, symbol device:D_Schottky
- added D? (x2): LED, symbol device:LED
- added J?: Conn_02x03_Odd_Even, symbol Connector:Conn_02x03_Odd_Even
- added R? (x2): 200, symbol device:R
- added R?: 10k, symbol device:R
- added U? (x7): 4050, symbol Logic_CMOS_4000:4050
Connections:
- net labels added: +5V, MISO1, MOSI1, RESET, SCK1, SS
- wire segments 61 -> 155
Other:
- moved on the sheet: J?

Commit message: Added the thermocouple module.
Parts:
- removed C? (x2): 14pF, symbol device:C
- removed Y?: 32.768KHz, symbol device:Crystal
- added R? (x3): 10k, symbol device:R
Connections:
- net labels added: CM, CS1, CS2, CS3, CS4, CS5, DA, DB, DC, DD, DRDY1, DRDY2, DRDY3, DRDY4, FAULT1, FAULT2, FAULT3, FAULT4, MISO2, MOSI2, SC, SCK2
- net labels removed: SS
- wire segments 155 -> 175

Commit message: Added switches
Parts:
- added C?: 0.1uF, symbol device:C
- added D?: D_Schottky, symbol device:D_Schottky
- added R?: 200, symbol device:R
- added R? (x2): 10k, symbol device:R
- R? (x3): value 10k -> 470k
- SW?: value SW_Push -> Reset
- gave numbers to parts that had none: 1
Connections:
- net labels added: DEBUG
- wire segments 175 -> 195
Other:
- moved on the sheet: U1

Commit message: Finished basic schimatic layout
Parts:
- J?: value Conn_02x03_Odd_Even -> ISP
- gave numbers to parts that had none: 1
Connections:
- net labels added: RCLK, SER, SRCLK
- net labels removed: DA, DB, DC
- wire segments 195 -> 202
Changed lines of the file:
@@
 F3 "Select/Calibrate" O L 9350 1550 50
 F4 "Cycle/Menu" O L 9350 1450 50
+F5 "SER" I L 9350 1100 50
+F6 "SRCLK" I L 9350 1200 50
+F7 "RCLK" I L 9350 1300 50
 $EndSheet
 $Comp
@@
 P 9600 3300
 F 0 "J?" H 9650 3617 50  0000 C CNN
-F 1 "Conn_02x03_Odd_Even" H 9650 3526 50  0000 C CNN
+F 1 "ISP" H 9650 3526 50  0000 C CNN
 F 2 "" H 9600 3300 50  0001 C CNN
 F 3 "~" H 9600 3300 50  0001 C CNN
@@
 RESET
 $Comp
-L Logic_CMOS_4000:4050 U?
+L Logic_CMOS_4000:4050 U14
 U 7 1 5A9A0A2A
 P 7150 3350
-F 0 "U?" H 7380 3396 50  0000 L CNN
+F 0 "U14" H 7380 3396 50  0000 L CNN
 F 1 "4050" H 7380 3305 50  0000 L CNN
 F 2 "" H 7150 3350 50  0001 C CNN
@@
 $EndComp
 $Comp
-L Logic_CMOS_4000:4050 U?
+L Logic_CMOS_4000:4050 U14
 U 1 1 5A9A89DB
 P 10400 3300
-F 0 "U?" H 10400 3617 50  0000 C CNN
+F 0 "U14" H 10400 3617 50  0000 C CNN
 F 1 "4050" H 10400 3526 50  0000 C CNN
 F 2 "" H 10400 3300 50  0001 C CNN
@@
 $EndComp
 $Comp
-L Logic_CMOS_4000:4050 U?
+L Logic_CMOS_4000:4050 U14
 U 2 1 5A9A8A59
 P 8800 3300
-F 0 "U?" H 8800 2983 50  0000 C CNN
+F 0 "U14" H 8800 2983 50  0000 C CNN
 F 1 "4050" H 8800 3074 50  0000 C CNN
 F 2 "" H 8800 3300 50  0001 C CNN
@@
 $EndComp
 $Comp
-L Logic_CMOS_4000:4050 U?
+L Logic_CMOS_4000:4050 U14
 U 3 1 5A9A8ADB
 P 8800 3900
-F 0 "U?" H 8800 3583 50  0000 C CNN
+F 0 "U14" H 8800 3583 50  0000 C CNN
 F 1 "4050" H 8800 3674 50  0000 C CNN
 F 2 "" H 8800 3900 50  0001 C CNN
@@
 	7150 4000 7150 3850
 $Comp
-L Logic_CMOS_4000:4050 U?
+L Logic_CMOS_4000:4050 U14
 U 4 1 5A9AAE84
 P 7500 5250
-F 0 "U?" H 7500 5567 50  0000 C CNN
+F 0 "U14" H 7500 5567 50  0000 C CNN
 F 1 "4050" H 7500 5476 50  0000 C CNN
 F 2 "" H 7500 5250 50  0001 C CNN
@@
 $EndComp
 $Comp
-L Logic_CMOS_4000:4050 U?
+L Logic_CMOS_4000:4050 U14
 U 5 1 5A9AAF0E
 P 7500 5750
-F 0 "U?" H 7500 6067 50  0000 C CNN
+F 0 "U14" H 7500 6067 50  0000 C CNN
 F 1 "4050" H 7500 5976 50  0000 C CNN
 F 2 "" H 7500 5750 50  0001 C CNN
@@
 $EndComp
 $Comp
-L Logic_CMOS_4000:4050 U?
+L Logic_CMOS_4000:4050 U14
 U 6 1 5A9AAF9E
 P 7500 4750
-F 0 "U?" H 7500 5067 50  0000 C CNN
+F 0 "U14" H 7500 5067 50  0000 C CNN
 F 1 "4050" H 7500 4976 50  0000 C CNN
 F 2 "" H 7500 4750 50  0001 C CNN
@@
 	4450 3850 4450 4050
 Text GLabel 4300 4350 2    50   Input ~ 0
-DA
+SER
 Text GLabel 4300 4450 2    50   Input ~ 0
-DB
+SRCLK
 Text GLabel 4300 4550 2    50   Input ~ 0
-DC
+RCLK
 Wire Wire Line
 	4000 4450 4300 4450
@@
 Wire Wire Line
 	4000 4650 4300 4650
-Text GLabel 4200 6350 2    50   Input ~ 0
+Text GLabel 4200 6450 2    50   Input ~ 0
 MOSI2
 $Sheet
@@
 Wire Wire Line
 	4200 6000 4550 6000
-Text GLabel 4200 6450 2    50   Input ~ 0
+Text GLabel 4200 6350 2    50   Input ~ 0
 MISO2
 Text GLabel 4200 6550 2    50   Input ~ 0
@@
 Connection ~ 8450 950
 Wire Wire Line
-	8450 950  9350 950
+	8450 950  8950 950
 Wire Wire Line
 	8450 1350 8450 1300
@@
 Wire Wire Line
 	9150 1550 9350 1550
+Wire Wire Line
+	4000 6350 4200 6350
+Wire Wire Line
+	4000 6450 4200 6450
+Text GLabel 9150 1100 0    50   Input ~ 0
+SER
+Text GLabel 9150 1200 0    50   Input ~ 0
+SRCLK
+Text GLabel 9150 1300 0    50   Input ~ 0
+RCLK
+Wire Wire Line
+	9150 1100 9350 1100
+Wire Wire Line
+	9150 1200 9350 1200
+Wire Wire Line
+	9150 1300 9350 1300
+Text GLabel 8950 800  1    50   Input ~ 0
+DD
+Wire Wire Line
+	8950 950  8950 800
+Connection ~ 8950 950
+Wire Wire Line
+	8950 950  9350 950
 $EndSCHEMATC

Commit message: Updated SD card slot to generic
Parts:
- removed J?: Micro_SD_Card_Det_Hirose_DM3AT, symbol Connector:Micro_SD_Card_Det_Hirose_DM3AT
- added J?: Micro_SD_Card_Det, symbol Connector:Micro_SD_Card_Det
Changed lines of the file:
@@
-	1    0    0    -1
-$EndComp
-$Comp
-L Connector:Micro_SD_Card_Det_Hirose_DM3AT J?
-U 1 1 5A862BAF
-P 10000 5450
-F 0 "J?" H 9950 6267 50  0000 C CNN
-F 1 "Micro_SD_Card_Det_Hirose_DM3AT" H 9950 6176 50  0000 C CNN
-F 2 "" H 12050 6150 50  0001 C CNN
-F 3 "https://www.hirose.com/product/en/download_file/key_name/DM3/category/Catalog/doc_file_id/49662/?file_category_id=4&item_id=195&is_series=1" H 10000 5550 50  0001 C CNN
-	1    10000 5450
 	1    0    0    -1
 $EndComp
@@
 Wire Wire Line
 	8950 950  9350 950
+$Comp
+L Connector:Micro_SD_Card_Det J?
+U 1 1 5A972AA1
+P 10000 5450
+F 0 "J?" H 9950 6267 50  0000 C CNN
+F 1 "Micro_SD_Card_Det" H 9950 6176 50  0000 C CNN
+F 2 "" H 12050 6150 50  0001 C CNN
+F 3 "https://www.hirose.com/product/en/download_file/key_name/DM3/category/Catalog/doc_file_id/49662/?file_category_id=4&item_id=195&is_series=1" H 10000 5550 50  0001 C CNN
+	1    10000 5450
+	1    0    0    -1
+$EndComp
 $EndSCHEMATC

Commit message: Annotated schematic
Parts:
- D0: renamed from D?; value LED -> Power
- D1: renamed from D?; value LED -> Debug
- SW1: renamed from SW?; value SW_SPDT -> Display
- gave numbers to parts that had none: 27
- renumbered U1 to U0, U14 to U13

Commit message: Renamed some components
Parts:
- D0: value Power -> LED Power
- D1: value Debug -> LED Debug
Changed lines of the file:
@@
 P 4700 3050
 F 0 "D0" H 4691 3266 50  0000 C CNN
-F 1 "Power" H 4691 3175 50  0000 C CNN
+F 1 "LED Power" H 4691 3175 50  0000 C CNN
 F 2 "" H 4700 3050 50  0001 C CNN
 F 3 "~" H 4700 3050 50  0001 C CNN
@@
 P 4650 4050
 F 0 "D1" H 4642 3795 50  0000 C CNN
-F 1 "Debug" H 4642 3886 50  0000 C CNN
+F 1 "LED Debug" H 4642 3886 50  0000 C CNN
 F 2 "" H 4650 4050 50  0001 C CNN
 F 3 "~" H 4650 4050 50  0001 C CNN

Commit message: Made footprint for the terminal block
Parts:
- C13, C14, C21, C22, C23, C24, C33, C34: footprint (none) -> Capacitors_SMD:C_0603
- C2, C3: footprint (none) -> Capacitors_SMD:C_0402
- D0, D1: footprint (none) -> LEDs:LED_0603
- D10, D11, D9: footprint (none) -> Diodes_SMD:D_SOD-323
- J1: footprint (none) -> Connectors_Card:Hirose_DM3BT-DSF-PEJS
- J6: footprint (none) -> Pin_Headers:Pin_Header_Straight_2x03_Pitch2.54mm
- U0: footprint VQFN44 -> (none)
Changed lines of the file:
@@
 F 0 "U0" H 3000 7400 50  0000 C CNN
 F 1 "ATMEGA324PA-MU" H 3000 7300 50  0000 C CNN
-F 2 "VQFN44" H 3000 5150 50  0001 C CIN
+F 2 "" H 3000 5150 50  0001 C CIN
 F 3 "http://www.atmel.com/Images/Atmel-8272-8-bit-AVR-microcontroller-ATmega164A_PA-324A_PA-644A_PA-1284_P_datasheet.pdf" H 3000 5150 50  0001 C CNN
 	1    3000 5150
@@
 F 0 "C24" V 3448 2900 50  0000 C CNN
 F 1 "0.33uF" V 3539 2900 50  0000 C CNN
-F 2 "" H 3738 2750 50  0001 C CNN
+F 2 "Capacitors_SMD:C_0603" H 3738 2750 50  0001 C CNN
 F 3 "" H 3700 2900 50  0001 C CNN
 	1    3700 2900
@@
 F 0 "C21" V 1898 2900 50  0000 C CNN
 F 1 "0.33uF" V 1989 2900 50  0000 C CNN
-F 2 "" H 2188 2750 50  0001 C CNN
+F 2 "Capacitors_SMD:C_0603" H 2188 2750 50  0001 C CNN
 F 3 "" H 2150 2900 50  0001 C CNN
 	1    2150 2900
@@
 F 0 "C22" V 2398 2400 50  0000 C CNN
 F 1 "0.33uF" V 2489 2400 50  0000 C CNN
-F 2 "" H 2688 2250 50  0001 C CNN
+F 2 "Capacitors_SMD:C_0603" H 2688 2250 50  0001 C CNN
 F 3 "" H 2650 2400 50  0001 C CNN
 	1    2650 2400
@@
 F 0 "C23" V 2948 2400 50  0000 C CNN
 F 1 "0.33uF" V 3039 2400 50  0000 C CNN
-F 2 "" H 3238 2250 50  0001 C CNN
+F 2 "Capacitors_SMD:C_0603" H 3238 2250 50  0001 C CNN
 F 3 "" H 3200 2400 50  0001 C CNN
 	1    3200 2400
@@
 F 0 "C13" V 1598 5000 50  0000 C CNN
 F 1 "0.1uF" V 1689 5000 50  0000 C CNN
-F 2 "" H 1888 4850 50  0001 C CNN
+F 2 "Capacitors_SMD:C_0603" H 1888 4850 50  0001 C CNN
 F 3 "" H 1850 5000 50  0001 C CNN
 	1    1850 5000
@@
 F 0 "C2" V 948 3550 50  0000 C CNN
 F 1 "18pF" V 1039 3550 50  0000 C CNN
-F 2 "" H 1238 3400 50  0001 C CNN
+F 2 "Capacitors_SMD:C_0402" H 1238 3400 50  0001 C CNN
 F 3 "" H 1200 3550 50  0001 C CNN
 	1    1200 3550
@@
 F 0 "C3" V 948 4500 50  0000 C CNN
 F 1 "18pF" V 1039 4500 50  0000 C CNN
-F 2 "" H 1238 4350 50  0001 C CNN
+F 2 "Capacitors_SMD:C_0402" H 1238 4350 50  0001 C CNN
 F 3 "" H 1200 4500 50  0001 C CNN
 	1    1200 4500
@@
 F 0 "J6" H 9650 3617 50  0000 C CNN
 F 1 "ISP" H 9650 3526 50  0000 C CNN
-F 2 "" H 9600 3300 50  0001 C CNN
+F 2 "Pin_Headers:Pin_Header_Straight_2x03_Pitch2.54mm" H 9600 3300 50  0001 C CNN
 F 3 "~" H 9600 3300 50  0001 C CNN
 	1    9600 3300
@@
 F 0 "C33" V 7198 2750 50  0000 C CNN
 F 1 "0.33uF" V 7289 2750 50  0000 C CNN
-F 2 "" H 7488 2600 50  0001 C CNN
+F 2 "Capacitors_SMD:C_0603" H 7488 2600 50  0001 C CNN
 F 3 "" H 7450 2750 50  0001 C CNN
 	1    7450 2750
@@
 F 0 "D10" V 8554 2479 50  0000 L CNN
 F 1 "D_Schottky" V 8645 2479 50  0000 L CNN
-F 2 "" H 8600 2400 50  0001 C CNN
+F 2 "Diodes_SMD:D_SOD-323" H 8600 2400 50  0001 C CNN
 F 3 "" H 8600 2400 50  0001 C CNN
 	1    8600 2400
@@
 F 0 "D9" V 8554 2179 50  0000 L CNN
 F 1 "D_Schottky" V 8645 2179 50  0000 L CNN
-F 2 "" H 8600 2100 50  0001 C CNN
+F 2 "Diodes_SMD:D_SOD-323" H 8600 2100 50  0001 C CNN
 F 3 "" H 8600 2100 50  0001 C CNN
 	1    8600 2100
@@
 F 0 "C34" V 8048 5500 50  0000 C CNN
 F 1 "0.33uF" V 8139 5500 50  0000 C CNN
-F 2 "" H 8338 5350 50  0001 C CNN
+F 2 "Capacitors_SMD:C_0603" H 8338 5350 50  0001 C CNN
 F 3 "" H 8300 5500 50  0001 C CNN
 	1    8300 5500
@@
 F 0 "D0" H 4691 3266 50  0000 C CNN
 F 1 "LED Power" H 4691 3175 50  0000 C CNN
-F 2 "" H 4700 3050 50  0001 C CNN
+F 2 "LEDs:LED_0603" H 4700 3050 50  0001 C CNN
 F 3 "~" H 4700 3050 50  0001 C CNN
 	1    4700 3050
@@
 F 0 "D1" H 4642 3795 50  0000 C CNN
 F 1 "LED Debug" H 4642 3886 50  0000 C CNN
-F 2 "" H 4650 4050 50  0001 C CNN
+F 2 "LEDs:LED_0603" H 4650 4050 50  0001 C CNN
 F 3 "~" H 4650 4050 50  0001 C CNN
 	1    4650 4050
@@
 F 0 "C14" V 5598 1550 50  0000 C CNN
 F 1 "0.1uF" V 5689 1550 50  0000 C CNN
-F 2 "" H 5888 1400 50  0001 C CNN
+F 2 "Capacitors_SMD:C_0603" H 5888 1400 50  0001 C CNN
 F 3 "" H 5850 1550 50  0001 C CNN
 	1    5850 1550
@@
 F 0 "D11" V 6154 1129 50  0000 L CNN
 F 1 "D_Schottky" V 6245 1129 50  0000 L CNN
-F 2 "" H 6200 1050 50  0001 C CNN
+F 2 "Diodes_SMD:D_SOD-323" H 6200 1050 50  0001 C CNN
 F 3 "" H 6200 1050 50  0001 C CNN
 	1    6200 1050
@@
 F 0 "J1" H 9950 6267 50  0000 C CNN
 F 1 "Micro_SD_Card_Det" H 9950 6176 50  0000 C CNN
-F 2 "" H 12050 6150 50  0001 C CNN
+F 2 "Connectors_Card:Hirose_DM3BT-DSF-PEJS" H 12050 6150 50  0001 C CNN
 F 3 "https://www.hirose.com/product/en/download_file/key_name/DM3/category/Catalog/doc_file_id/49662/?file_category_id=4&item_id=195&is_series=1" H 10000 5550 50  0001 C CNN
 	1    10000 5450
