File: Thermocouple-Data-Logger/Thermocouple Data Logger.sch (KiCad schematic (older format))
At the start: 32 parts, among them J1 Micro_SD_Card_Det, J6 ISP, SW1 Display, SW2 Reset, SW5 SW_DIP_x04, U0 ATMEGA324PA-MU, U13 4050, Y0 10MHz

Commit message: Added the components and generaterd the netlist
Parts:
- R10, R8, R9: footprint (none) -> Resistors_SMD:R_0805
- R52, R53, R54, R57, R58, R59: footprint (none) -> Resistors_SMD:R_0402
- SW1: footprint (none) -> Buttons_Switches_SMD:SW_SPDT_CK-JS102011SAQN
- SW2: footprint (none) -> Buttons_Switches_SMD:SW_SPST_PTS645
- SW5: footprint (none) -> Buttons_Switches_SMD:SW_DIP_x4_W5.08mm_Slide_Copal_CHS-A
- U0: footprint (none) -> Housings_DFN_QFN:QFN-44-1EP_7x7mm_Pitch0.5mm
- U13: footprint (none) -> Housings_SSOP:TSSOP-16_4.4x5mm_Pitch0.65mm
- Y0: footprint (none) -> Crystals:Crystal_SMD_Abracon_ABM3B-4pin_5.0x3.2mm
Changed lines of the file:
@@
 F 0 "U0" H 3000 7400 50  0000 C CNN
 F 1 "ATMEGA324PA-MU" H 3000 7300 50  0000 C CNN
-F 2 "" H 3000 5150 50  0001 C CIN
+F 2 "Housings_DFN_QFN:QFN-44-1EP_7x7mm_Pitch0.5mm" H 3000 5150 50  0001 C CIN
 F 3 "http://www.atmel.com/Images/Atmel-8272-8-bit-AVR-microcontroller-ATmega164A_PA-324A_PA-644A_PA-1284_P_datasheet.pdf" H 3000 5150 50  0001 C CNN
 	1    3000 5150
@@
 F 0 "SW1" H 8200 1135 50  0000 C CNN
 F 1 "Display" H 8200 1044 50  0000 C CNN
-F 2 "" H 8200 850 50  0001 C CNN
+F 2 "Buttons_Switches_SMD:SW_SPDT_CK-JS102011SAQN" H 8200 850 50  0001 C CNN
 F 3 "" H 8200 850 50  0001 C CNN
 	1    8200 850
@@
 F 0 "SW5" H 4700 2967 50  0000 C CNN
 F 1 "SW_DIP_x04" H 4700 2876 50  0000 C CNN
-F 2 "" H 4700 2500 50  0001 C CNN
+F 2 "Buttons_Switches_SMD:SW_DIP_x4_W5.08mm_Slide_Copal_CHS-A" H 4700 2500 50  0001 C CNN
 F 3 "" H 4700 2500 50  0001 C CNN
 	1    4700 2500
@@
 F 0 "SW2" H 5100 1585 50  0000 C CNN
 F 1 "Reset" H 5100 1494 50  0000 C CNN
-F 2 "" H 5100 1500 50  0001 C CNN
+F 2 "Buttons_Switches_SMD:SW_SPST_PTS645" H 5100 1500 50  0001 C CNN
 F 3 "" H 5100 1500 50  0001 C CNN
 	1    5100 1300
@@
 F 0 "Y0" V 1100 3700 50  0000 L CNN
 F 1 "10MHz" V 1200 3700 50  0000 L CNN
-F 2 "" H 1400 4050 50  0001 C CNN
+F 2 "Crystals:Crystal_SMD_Abracon_ABM3B-4pin_5.0x3.2mm" H 1400 4050 50  0001 C CNN
 F 3 "" H 1400 4050 50  0001 C CNN
 	1    1400 4050
@@
 F 0 "U13" H 7380 3396 50  0000 L CNN
 F 1 "4050" H 7380 3305 50  0000 L CNN
-F 2 "" H 7150 3350 50  0001 C CNN
+F 2 "Housings_SSOP:TSSOP-16_4.4x5mm_Pitch0.65mm" H 7150 3350 50  0001 C CNN
 F 3 "http://www.intersil.com/content/dam/intersil/documents/cd40/cd4050bms.pdf" H 7150 3350 50  0001 C CNN
 	7    7150 3350
@@
 F 0 "U13" H 10400 3617 50  0000 C CNN
 F 1 "4050" H 10400 3526 50  0000 C CNN
-F 2 "" H 10400 3300 50  0001 C CNN
+F 2 "Housings_SSOP:TSSOP-16_4.4x5mm_Pitch0.65mm" H 10400 3300 50  0001 C CNN
 F 3 "http://www.intersil.com/content/dam/intersil/documents/cd40/cd4050bms.pdf" H 10400 3300 50  0001 C CNN
 	1    10400 3300
@@
 F 0 "U13" H 8800 2983 50  0000 C CNN
 F 1 "4050" H 8800 3074 50  0000 C CNN
-F 2 "" H 8800 3300 50  0001 C CNN
+F 2 "Housings_SSOP:TSSOP-16_4.4x5mm_Pitch0.65mm" H 8800 3300 50  0001 C CNN
 F 3 "http://www.intersil.com/content/dam/intersil/documents/cd40/cd4050bms.pdf" H 8800 3300 50  0001 C CNN
 	2    8800 3300
@@
 F 0 "U13" H 8800 3583 50  0000 C CNN
 F 1 "4050" H 8800 3674 50  0000 C CNN
-F 2 "" H 8800 3900 50  0001 C CNN
+F 2 "Housings_SSOP:TSSOP-16_4.4x5mm_Pitch0.65mm" H 8800 3900 50  0001 C CNN
 F 3 "http://www.intersil.com/content/dam/intersil/documents/cd40/cd4050bms.pdf" H 8800 3900 50  0001 C CNN
 	3    8800 3900
@@
 F 0 "U13" H 7500 5567 50  0000 C CNN
 F 1 "4050" H 7500 5476 50  0000 C CNN
-F 2 "" H 7500 5250 50  0001 C CNN
+F 2 "Housings_SSOP:TSSOP-16_4.4x5mm_Pitch0.65mm" H 7500 5250 50  0001 C CNN
 F 3 "http://www.intersil.com/content/dam/intersil/documents/cd40/cd4050bms.pdf" H 7500 5250 50  0001 C CNN
 	4    7500 5250
@@
 F 0 "U13" H 7500 6067 50  0000 C CNN
 F 1 "4050" H 7500 5976 50  0000 C CNN
-F 2 "" H 7500 5750 50  0001 C CNN
+F 2 "Housings_SSOP:TSSOP-16_4.4x5mm_Pitch0.65mm" H 7500 5750 50  0001 C CNN
 F 3 "http://www.intersil.com/content/dam/intersil/documents/cd40/cd4050bms.pdf" H 7500 5750 50  0001 C CNN
 	5    7500 5750
@@
 F 0 "U13" H 7500 5067 50  0000 C CNN
 F 1 "4050" H 7500 4976 50  0000 C CNN
-F 2 "" H 7500 4750 50  0001 C CNN
+F 2 "Housings_SSOP:TSSOP-16_4.4x5mm_Pitch0.65mm" H 7500 4750 50  0001 C CNN
 F 3 "http://www.intersil.com/content/dam/intersil/documents/cd40/cd4050bms.pdf" H 7500 4750 50  0001 C CNN
 	6    7500 4750
@@
 F 0 "R8" H 4320 2946 50  0000 L CNN
 F 1 "200" H 4320 2855 50  0000 L CNN
-F 2 "" V 4180 2900 50  0001 C CNN
+F 2 "Resistors_SMD:R_0805" V 4180 2900 50  0001 C CNN
 F 3 "" H 4250 2900 50  0001 C CNN
 	1    4250 2900
@@
 F 0 "R52" V 4493 3350 50  0000 C CNN
 F 1 "10k" V 4584 3350 50  0000 C CNN
-F 2 "" V 4630 3350 50  0001 C CNN
+F 2 "Resistors_SMD:R_0402" V 4630 3350 50  0001 C CNN
 F 3 "" H 4700 3350 50  0001 C CNN
 	1    4700 3350
@@
 F 0 "R10" V 5207 4050 50  0000 C CNN
 F 1 "200" V 5116 4050 50  0000 C CNN
-F 2 "" V 4930 4050 50  0001 C CNN
+F 2 "Resistors_SMD:R_0805" V 4930 4050 50  0001 C CNN
 F 3 "" H 5000 4050 50  0001 C CNN
 	1    5000 4050
@@
 F 0 "R57" V 5693 2300 50  0000 C CNN
 F 1 "470k" V 5784 2300 50  0000 C CNN
-F 2 "" V 5830 2300 50  0001 C CNN
+F 2 "Resistors_SMD:R_0402" V 5830 2300 50  0001 C CNN
 F 3 "" H 5900 2300 50  0001 C CNN
 	1    5900 2300
@@
 F 0 "R58" V 5693 2600 50  0000 C CNN
 F 1 "470k" V 5784 2600 50  0000 C CNN
-F 2 "" V 5830 2600 50  0001 C CNN
+F 2 "Resistors_SMD:R_0402" V 5830 2600 50  0001 C CNN
 F 3 "" H 5900 2600 50  0001 C CNN
 	1    5900 2600
@@
 F 0 "R59" V 5693 2900 50  0000 C CNN
 F 1 "470k" V 5784 2900 50  0000 C CNN
-F 2 "" V 5830 2900 50  0001 C CNN
+F 2 "Resistors_SMD:R_0402" V 5830 2900 50  0001 C CNN
 F 3 "" H 5900 2900 50  0001 C CNN
 	1    5900 2900
@@
 F 0 "R54" V 8243 1150 50  0000 C CNN
 F 1 "10k" V 8334 1150 50  0000 C CNN
-F 2 "" V 8380 1150 50  0001 C CNN
+F 2 "Resistors_SMD:R_0402" V 8380 1150 50  0001 C CNN
 F 3 "" H 8450 1150 50  0001 C CNN
 	1    8450 1150
@@
 F 0 "R53" V 5643 1050 50  0000 C CNN
 F 1 "10k" V 5734 1050 50  0000 C CNN
-F 2 "" V 5780 1050 50  0001 C CNN
+F 2 "Resistors_SMD:R_0402" V 5780 1050 50  0001 C CNN
 F 3 "" H 5850 1050 50  0001 C CNN
 	1    5850 1050
@@
 F 0 "R9" H 5620 1346 50  0000 L CNN
 F 1 "200" H 5620 1255 50  0000 L CNN
-F 2 "" V 5480 1300 50  0001 C CNN
+F 2 "Resistors_SMD:R_0805" V 5480 1300 50  0001 C CNN
 F 3 "" H 5550 1300 50  0001 C CNN
 	1    5550 1300

Commit message: Added mounting holes, grounding holes and fiducials
Changed lines of the file:
@@
 $Descr A4 11693 8268
 encoding utf-8
-Sheet 1 5
+Sheet 1 6
 Title ""
 Date ""
@@
 	1    0    0    -1
 $EndComp
+$Sheet
+S 2550 800  950  550
+U 5A9A89AB
+F0 "Mounting_Hole" 50
+F1 "Mounting_Hole.sch" 50
+$EndSheet
 $EndSCHEMATC

Commit message: Changed capacitor values and component layout
Parts:
- C17: renamed from C13; footprint Capacitors_SMD:C_0603 -> Capacitors_SMD:C_0402
- C18: renamed from C14; footprint Capacitors_SMD:C_0603 -> Capacitors_SMD:C_0402
- C21, C22, C23, C24, C33, C34: value 0.33uF -> 0.1uF; footprint Capacitors_SMD:C_0603 -> Capacitors_SMD:C_0402
Changed lines of the file:
@@
 P 3700 2900
 F 0 "C24" V 3448 2900 50  0000 C CNN
-F 1 "0.33uF" V 3539 2900 50  0000 C CNN
-F 2 "Capacitors_SMD:C_0603" H 3738 2750 50  0001 C CNN
+F 1 "0.1uF" V 3539 2900 50  0000 C CNN
+F 2 "Capacitors_SMD:C_0402" H 3738 2750 50  0001 C CNN
 F 3 "" H 3700 2900 50  0001 C CNN
 	1    3700 2900
@@
 P 2150 2900
 F 0 "C21" V 1898 2900 50  0000 C CNN
-F 1 "0.33uF" V 1989 2900 50  0000 C CNN
-F 2 "Capacitors_SMD:C_0603" H 2188 2750 50  0001 C CNN
+F 1 "0.1uF" V 1989 2900 50  0000 C CNN
+F 2 "Capacitors_SMD:C_0402" H 2188 2750 50  0001 C CNN
 F 3 "" H 2150 2900 50  0001 C CNN
 	1    2150 2900
@@
 P 2650 2400
 F 0 "C22" V 2398 2400 50  0000 C CNN
-F 1 "0.33uF" V 2489 2400 50  0000 C CNN
-F 2 "Capacitors_SMD:C_0603" H 2688 2250 50  0001 C CNN
+F 1 "0.1uF" V 2489 2400 50  0000 C CNN
+F 2 "Capacitors_SMD:C_0402" H 2688 2250 50  0001 C CNN
 F 3 "" H 2650 2400 50  0001 C CNN
 	1    2650 2400
@@
 P 3200 2400
 F 0 "C23" V 2948 2400 50  0000 C CNN
-F 1 "0.33uF" V 3039 2400 50  0000 C CNN
-F 2 "Capacitors_SMD:C_0603" H 3238 2250 50  0001 C CNN
+F 1 "0.1uF" V 3039 2400 50  0000 C CNN
+F 2 "Capacitors_SMD:C_0402" H 3238 2250 50  0001 C CNN
 F 3 "" H 3200 2400 50  0001 C CNN
 	1    3200 2400
@@
 	2000 3000 2000 2900
 $Comp
-L device:C C13
+L device:C C17
 U 1 1 5A8EC7BC
 P 1850 5000
-F 0 "C13" V 1598 5000 50  0000 C CNN
+F 0 "C17" V 1598 5000 50  0000 C CNN
 F 1 "0.1uF" V 1689 5000 50  0000 C CNN
-F 2 "Capacitors_SMD:C_0603" H 1888 4850 50  0001 C CNN
+F 2 "Capacitors_SMD:C_0402" H 1888 4850 50  0001 C CNN
 F 3 "" H 1850 5000 50  0001 C CNN
 	1    1850 5000
@@
 P 7450 2750
 F 0 "C33" V 7198 2750 50  0000 C CNN
-F 1 "0.33uF" V 7289 2750 50  0000 C CNN
-F 2 "Capacitors_SMD:C_0603" H 7488 2600 50  0001 C CNN
+F 1 "0.1uF" V 7289 2750 50  0000 C CNN
+F 2 "Capacitors_SMD:C_0402" H 7488 2600 50  0001 C CNN
 F 3 "" H 7450 2750 50  0001 C CNN
 	1    7450 2750
@@
 P 8300 5500
 F 0 "C34" V 8048 5500 50  0000 C CNN
-F 1 "0.33uF" V 8139 5500 50  0000 C CNN
-F 2 "Capacitors_SMD:C_0603" H 8338 5350 50  0001 C CNN
+F 1 "0.1uF" V 8139 5500 50  0000 C CNN
+F 2 "Capacitors_SMD:C_0402" H 8338 5350 50  0001 C CNN
 F 3 "" H 8300 5500 50  0001 C CNN
 	1    8300 5500
@@
 	4750 1300 4900 1300
 $Comp
-L device:C C14
+L device:C C18
 U 1 1 5ADC93BA
 P 5850 1550
-F 0 "C14" V 5598 1550 50  0000 C CNN
+F 0 "C18" V 5598 1550 50  0000 C CNN
 F 1 "0.1uF" V 5689 1550 50  0000 C CNN
-F 2 "Capacitors_SMD:C_0603" H 5888 1400 50  0001 C CNN
+F 2 "Capacitors_SMD:C_0402" H 5888 1400 50  0001 C CNN
 F 3 "" H 5850 1550 50  0001 C CNN
 	1    5850 1550

Commit message: Finished routing all traces
Connections:
- wire segments 202 -> 201
Changed lines of the file:
@@
 	5600 4100 5650 4100
-Wire Wire Line
-	5650 4100 5650 4200
 Wire Wire Line
 	5650 4200 5600 4200

Commit message: Changed the microcontroller from qfn to tqfp
Parts:
- C17, C18, C2, C21, C22, C23, C24, C3, C33, C34: symbol device:C -> Thermocouple-Data-Logger-rescue:C-device
- D0, D1: symbol device:LED -> Thermocouple-Data-Logger-rescue:LED-device
- D10, D11, D9: symbol device:D_Schottky -> Thermocouple-Data-Logger-rescue:D_Schottky-device
- J1: symbol Connector:Micro_SD_Card_Det -> Thermocouple-Data-Logger-rescue:Micro_SD_Card_Det-Connector
- J6: symbol Connector:Conn_02x03_Odd_Even -> Thermocouple-Data-Logger-rescue:Conn_02x03_Odd_Even-Connector
- R10, R52, R53, R54, R57, R58, R59, R8, R9: symbol device:R -> Thermocouple-Data-Logger-rescue:R-device
- U0: footprint Housings_DFN_QFN:QFN-44-1EP_7x7mm_Pitch0.5mm -> Housings_QFP:TQFP-44_10x10mm_Pitch0.8mm; symbol atmel:ATMEGA324PA-MU -> Thermocouple-Data-Logger-rescue:ATMEGA324PA-MU-atmel
- U13: symbol Logic_CMOS_4000:4050 -> Thermocouple-Data-Logger-rescue:4050-Logic_CMOS_4000
- Y0: symbol device:Crystal_GND24 -> Thermocouple-Data-Logger-rescue:Crystal_GND24-device
Changed lines of the file:
@@
 $EndDescr
 $Comp
-L atmel:ATMEGA324PA-MU U0
+L Thermocouple-Data-Logger-rescue:ATMEGA324PA-MU-atmel U0
 U 1 1 5A8617D1
 P 3000 5150
 F 0 "U0" H 3000 7400 50  0000 C CNN
 F 1 "ATMEGA324PA-MU" H 3000 7300 50  0000 C CNN
-F 2 "Housings_DFN_QFN:QFN-44-1EP_7x7mm_Pitch0.5mm" H 3000 5150 50  0001 C CIN
+F 2 "Housings_QFP:TQFP-44_10x10mm_Pitch0.8mm" H 3000 5150 50  0001 C CIN
 F 3 "http://www.atmel.com/Images/Atmel-8272-8-bit-AVR-microcontroller-ATmega164A_PA-324A_PA-644A_PA-1284_P_datasheet.pdf" H 3000 5150 50  0001 C CNN
 	1    3000 5150
@@
 	2800 7300 2850 7300
 $Comp
-L device:C C24
+L Thermocouple-Data-Logger-rescue:C-device C24
 U 1 1 5A8E6FD1
 P 3700 2900
@@
 $EndComp
 $Comp
-L device:C C21
+L Thermocouple-Data-Logger-rescue:C-device C21
 U 1 1 5A8E7D56
 P 2150 2900
@@
 $EndComp
 $Comp
-L device:C C22
+L Thermocouple-Data-Logger-rescue:C-device C22
 U 1 1 5A8E7D82
 P 2650 2400
@@
 $EndComp
 $Comp
-L device:C C23
+L Thermocouple-Data-Logger-rescue:C-device C23
 U 1 1 5A8E7DB2
 P 3200 2400
@@
 	2000 3000 2000 2900
 $Comp
-L device:C C17
+L Thermocouple-Data-Logger-rescue:C-device C17
 U 1 1 5A8EC7BC
 P 1850 5000
@@
 	1350 5000 1700 5000
 $Comp
-L device:Crystal_GND24 Y0
+L Thermocouple-Data-Logger-rescue:Crystal_GND24-device Y0
 U 1 1 5A8F2265
 P 1400 4050
@@
 	4200 5950 4200 6000
 $Comp
-L device:C C2
+L Thermocouple-Data-Logger-rescue:C-device C2
 U 1 1 5A8FCA8F
 P 1200 3550
@@
 $EndComp
 $Comp
-L device:C C3
+L Thermocouple-Data-Logger-rescue:C-device C3
 U 1 1 5A8FCCFB
 P 1200 4500
@@
 $EndComp
 $Comp
-L Connector:Conn_02x03_Odd_Even J6
+L Thermocouple-Data-Logger-rescue:Conn_02x03_Odd_Even-Connector J6
 U 1 1 5A984B5E
 P 9600 3300
@@
 RESET
 $Comp
-L Logic_CMOS_4000:4050 U13
+L Thermocouple-Data-Logger-rescue:4050-Logic_CMOS_4000 U13
 U 7 1 5A9A0A2A
 P 7150 3350
@@
 $EndComp
 $Comp
-L Logic_CMOS_4000:4050 U13
+L Thermocouple-Data-Logger-rescue:4050-Logic_CMOS_4000 U13
 U 1 1 5A9A89DB
 P 10400 3300
@@
 $EndComp
 $Comp
-L Logic_CMOS_4000:4050 U13
+L Thermocouple-Data-Logger-rescue:4050-Logic_CMOS_4000 U13
 U 2 1 5A9A8A59
 P 8800 3300
@@
 $EndComp
 $Comp
-L Logic_CMOS_4000:4050 U13
+L Thermocouple-Data-Logger-rescue:4050-Logic_CMOS_4000 U13
 U 3 1 5A9A8ADB
 P 8800 3900
@@
 	7150 4000 7150 3850
 $Comp
-L Logic_CMOS_4000:4050 U13
+L Thermocouple-Data-Logger-rescue:4050-Logic_CMOS_4000 U13
 U 4 1 5A9AAE84
 P 7500 5250
@@
 $EndComp
 $Comp
-L Logic_CMOS_4000:4050 U13
+L Thermocouple-Data-Logger-rescue:4050-Logic_CMOS_4000 U13
 U 5 1 5A9AAF0E
 P 7500 5750
@@
 $EndComp
 $Comp
-L Logic_CMOS_4000:4050 U13
+L Thermocouple-Data-Logger-rescue:4050-Logic_CMOS_4000 U13
 U 6 1 5A9AAF9E
 P 7500 4750
@@
 	7150 2850 7150 2750
 $Comp
-L device:C C33
+L Thermocouple-Data-Logger-rescue:C-device C33
 U 1 1 5A9B9571
 P 7450 2750
@@
 $EndComp
 $Comp
-L device:D_Schottky D10
+L Thermocouple-Data-Logger-rescue:D_Schottky-device D10
 U 1 1 5A9F17B2
 P 8600 2400
@@
 $EndComp
 $Comp
-L device:D_Schottky D9
+L Thermocouple-Data-Logger-rescue:D_Schottky-device D9
 U 1 1 5A9F182D
 P 8600 2100
@@
 	8600 5650 8600 5550
 $Comp
-L device:C C34
+L Thermocouple-Data-Logger-rescue:C-device C34
 U 1 1 5AA11AA3
 P 8300 5500
@@
 	5050 3050 5050 2600
 $Comp
-L device:LED D0
+L Thermocouple-Data-Logger-rescue:LED-device D0
 U 1 1 5AA7B2DF
 P 4700 3050
@@
 $EndComp
 $Comp
-L device:R R8
+L Thermocouple-Data-Logger-rescue:R-device R8
 U 1 1 5AA8E8C6
 P 4250 2900
@@
 	5000 2600 5050 2600
 $Comp
-L device:R R52
+L Thermocouple-Data-Logger-rescue:R-device R52
 U 1 1 5AAD9464
 P 4700 3350
@@
 	5050 3350 5050 3050
 $Comp
-L device:LED D1
+L Thermocouple-Data-Logger-rescue:LED-device D1
 U 1 1 5AB14889
 P 4650 4050
@@
 Connection ~ 4250 3050
 $Comp
-L device:R R10
+L Thermocouple-Data-Logger-rescue:R-device R10
 U 1 1 5AB18F7F
 P 5000 4050
@@
 	5550 5400 5650 5400
 $Comp
-L device:R R57
+L Thermocouple-Data-Logger-rescue:R-device R57
 U 1 1 5AC32C62
 P 5900 2300
@@
 $EndComp
 $Comp
-L device:R R58
+L Thermocouple-Data-Logger-rescue:R-device R58
 U 1 1 5AC32CD0
 P 5900 2600
@@
 $EndComp
 $Comp
-L device:R R59
+L Thermocouple-Data-Logger-rescue:R-device R59
 U 1 1 5AC32D28
 P 5900 2900
@@
 	5150 2900 5150 3750
 $Comp
-L device:R R54
+L Thermocouple-Data-Logger-rescue:R-device R54
 U 1 1 5AC9C9C4
 P 8450 1150
@@
 	5850 1300 6200 1300
 $Comp
-L device:R R53
+L Thermocouple-Data-Logger-rescue:R-device R53
 U 1 1 5AD37429
 P 5850 1050
@@
 	4750 1300 4900 1300
 $Comp
-L device:C C18
+L Thermocouple-Data-Logger-rescue:C-device C18
 U 1 1 5ADC93BA
 P 5850 1550
@@
 DEBUG
 $Comp
-L device:D_Schottky D11
+L Thermocouple-Data-Logger-rescue:D_Schottky-device D11
 U 1 1 5A9A15D5
 P 6200 1050
@@
 	5850 850  5850 800
 $Comp
-L device:R R9
+L Thermocouple-Data-Logger-rescue:R-device R9
 U 1 1 5A9BE9D0
 P 5550 1300
@@
 	8950 950  9350 950
 $Comp
-L Connector:Micro_SD_Card_Det J1
+L Thermocouple-Data-Logger-rescue:Micro_SD_Card_Det-Connector J1
 U 1 1 5A972AA1
 P 10000 5450
