File: Thermocouple-Data-Logger/Display.sch (KiCad schematic (older format))
At the start: 16 parts

Commit message: Added switches
Parts:
- removed SW?: SW_Push, symbol Switch:SW_Push
- added C? (x2): 0.1uF, symbol device:C
- added R? (x2): 10k, symbol device:R
- added R? (x2): 1k, symbol device:R
- added SW?: Cycle/Menu, symbol Switch:SW_Push
- SW?: value SW_Push -> Select/Calibrate
- gave numbers to parts that had none: 5
Connections:
- net labels added: GND
- wire segments 4 -> 16
Changed lines of the file:
@@
 $EndDescr
 $Comp
-L Logic_74xx:74HC595 U?
+L Logic_74xx:74HC595 U7
 U 1 1 5A86784D
 P 2900 3500
-F 0 "U?" H 2900 4378 50  0000 C CNN
+F 0 "U7" H 2900 4378 50  0000 C CNN
 F 1 "74HC595" H 2900 4287 50  0000 C CNN
 F 2 "" H 2900 3500 50  0001 C CNN
@@
 $EndComp
 $Comp
-L Logic_74xx:74HC595 U?
+L Logic_74xx:74HC595 U8
 U 1 1 5A867854
 P 4300 3500
-F 0 "U?" H 4300 4378 50  0000 C CNN
+F 0 "U8" H 4300 4378 50  0000 C CNN
 F 1 "74HC595" H 4300 4287 50  0000 C CNN
 F 2 "" H 4300 3500 50  0001 C CNN
@@
 $EndComp
 $Comp
-L Logic_74xx:74HC595 U?
+L Logic_74xx:74HC595 U9
 U 1 1 5A86785B
 P 5650 3500
-F 0 "U?" H 5650 4378 50  0000 C CNN
+F 0 "U9" H 5650 4378 50  0000 C CNN
 F 1 "74HC595" H 5650 4287 50  0000 C CNN
 F 2 "" H 5650 3500 50  0001 C CNN
@@
 $EndComp
 $Comp
-L Logic_74xx:74HC595 U?
+L Logic_74xx:74HC595 U10
 U 1 1 5A867862
 P 6900 3500
-F 0 "U?" H 6900 4378 50  0000 C CNN
+F 0 "U10" H 6900 4378 50  0000 C CNN
 F 1 "74HC595" H 6900 4287 50  0000 C CNN
 F 2 "" H 6900 3500 50  0001 C CNN
@@
 VCC
 $Comp
-L Logic_74xx:74HC595 U?
+L Logic_74xx:74HC595 U11
 U 1 1 5A868ED4
 P 8250 3500
-F 0 "U?" H 8250 4378 50  0000 C CNN
+F 0 "U11" H 8250 4378 50  0000 C CNN
 F 1 "74HC595" H 8250 4287 50  0000 C CNN
 F 2 "" H 8250 3500 50  0001 C CNN
@@
 $Comp
 L Switch:SW_Push SW?
-U 1 1 5A8DCCD8
-P 2250 4850
-F 0 "SW?" H 2250 5135 50  0000 C CNN
-F 1 "SW_Push" H 2250 5044 50  0000 C CNN
-F 2 "" H 2250 5050 50  0001 C CNN
-F 3 "" H 2250 5050 50  0001 C CNN
-	1    2250 4850
-	1    0    0    -1
-$EndComp
-$Comp
-L Switch:SW_Push SW?
 U 1 1 5A8DCE11
-P 2300 5900
-F 0 "SW?" H 2300 6185 50  0000 C CNN
-F 1 "SW_Push" H 2300 6094 50  0000 C CNN
-F 2 "" H 2300 6100 50  0001 C CNN
-F 3 "" H 2300 6100 50  0001 C CNN
-	1    2300 5900
-	1    0    0    -1
-$EndComp
-Text HLabel 1750 4850 0    50   Output ~ 0
-Cycle/Menu
-Text HLabel 1700 5900 0    50   Output ~ 0
+P 2700 6500
+F 0 "SW?" H 2700 6785 50  0000 C CNN
+F 1 "Select/Calibrate" H 2700 6694 50  0000 C CNN
+F 2 "" H 2700 6700 50  0001 C CNN
+F 3 "" H 2700 6700 50  0001 C CNN
+	1    2700 6500
+	1    0    0    -1
+$EndComp
+Text HLabel 1650 6500 0    50   Output ~ 0
 Select/Calibrate
 Wire Wire Line
-	1750 4850 2050 4850
-Wire Wire Line
-	1700 5900 2100 5900
-Text HLabel 3100 4850 2    50   Input ~ 0
-VCC
-Text HLabel 3100 5900 2    50   Input ~ 0
-VCC
-Wire Wire Line
-	3100 4850 2450 4850
-Wire Wire Line
-	2500 5900 3100 5900
+	1650 6500 1900 6500
+Text HLabel 3050 6500 2    50   Input ~ 0
+VCC
+Wire Wire Line
+	2900 6500 3050 6500
 $Comp
 L Thermocouple-Data-Logger:HDSP-521E-Display U?
@@
 	1    0    0    -1
 $EndComp
+$Comp
+L device:R R?
+U 1 1 5AD8AEEC
+P 1900 6800
+F 0 "R?" V 1693 6800 50  0000 C CNN
+F 1 "10k" V 1784 6800 50  0000 C CNN
+F 2 "" V 1830 6800 50  0001 C CNN
+F 3 "" H 1900 6800 50  0001 C CNN
+	1    1900 6800
+	-1   0    0    1
+$EndComp
+$Comp
+L power:GND #PWR?
+U 1 1 5AD8AFB4
+P 1900 7100
+F 0 "#PWR?" H 1900 6850 50  0001 C CNN
+F 1 "GND" H 1905 6927 50  0000 C CNN
+F 2 "" H 1900 7100 50  0001 C CNN
+F 3 "" H 1900 7100 50  0001 C CNN
+	1    1900 7100
+	1    0    0    -1
+$EndComp
+Wire Wire Line
+	1900 7100 1900 6950
+Wire Wire Line
+	1900 6650 1900 6500
+Connection ~ 1900 6500
+$Comp
+L Switch:SW_Push SW?
+U 1 1 5AD8C388
+P 5600 6500
+F 0 "SW?" H 5600 6785 50  0000 C CNN
+F 1 "Cycle/Menu" H 5600 6694 50  0000 C CNN
+F 2 "" H 5600 6700 50  0001 C CNN
+F 3 "" H 5600 6700 50  0001 C CNN
+	1    5600 6500
+	1    0    0    -1
+$EndComp
+Text HLabel 4550 6500 0    50   Output ~ 0
+Cycle/Menu
+Wire Wire Line
+	4550 6500 4800 6500
+Text HLabel 5950 6500 2    50   Input ~ 0
+VCC
+Wire Wire Line
+	5800 6500 5950 6500
+$Comp
+L device:R R?
+U 1 1 5AD8C3A0
+P 4800 6800
+F 0 "R?" V 4593 6800 50  0000 C CNN
+F 1 "10k" V 4684 6800 50  0000 C CNN
+F 2 "" V 4730 6800 50  0001 C CNN
+F 3 "" H 4800 6800 50  0001 C CNN
+	1    4800 6800
+	-1   0    0    1
+$EndComp
+$Comp
+L power:GND #PWR?
+U 1 1 5AD8C3A7
+P 4800 7100
+F 0 "#PWR?" H 4800 6850 50  0001 C CNN
+F 1 "GND" H 4805 6927 50  0000 C CNN
+F 2 "" H 4800 7100 50  0001 C CNN
+F 3 "" H 4800 7100 50  0001 C CNN
+	1    4800 7100
+	1    0    0    -1
+$EndComp
+Wire Wire Line
+	4800 7100 4800 6950
+Wire Wire Line
+	4800 6650 4800 6500
+Connection ~ 4800 6500
+Wire Wire Line
+	4800 6500 5000 6500
+Wire Wire Line
+	1900 6500 2100 6500
+$Comp
+L device:C C?
+U 1 1 5ADBEA6C
+P 1900 6150
+F 0 "C?" H 2015 6196 50  0000 L CNN
+F 1 "0.1uF" H 2015 6105 50  0000 L CNN
+F 2 "" H 1938 6000 50  0001 C CNN
+F 3 "" H 1900 6150 50  0001 C CNN
+	1    1900 6150
+	1    0    0    -1
+$EndComp
+$Comp
+L device:C C?
+U 1 1 5ADBECAE
+P 4800 6150
+F 0 "C?" H 4915 6196 50  0000 L CNN
+F 1 "0.1uF" H 4915 6105 50  0000 L CNN
+F 2 "" H 4838 6000 50  0001 C CNN
+F 3 "" H 4800 6150 50  0001 C CNN
+	1    4800 6150
+	1    0    0    -1
+$EndComp
+Wire Wire Line
+	1900 6500 1900 6300
+Wire Wire Line
+	4800 6500 4800 6300
+Text HLabel 4800 5800 1    50   Input ~ 0
+VCC
+Text HLabel 1900 5800 1    50   Input ~ 0
+VCC
+Wire Wire Line
+	4800 6000 4800 5800
+Wire Wire Line
+	1900 6000 1900 5800
+$Comp
+L device:R R?
+U 1 1 5ADBF30B
+P 2250 6500
+F 0 "R?" V 2043 6500 50  0000 C CNN
+F 1 "1k" V 2134 6500 50  0000 C CNN
+F 2 "" V 2180 6500 50  0001 C CNN
+F 3 "" H 2250 6500 50  0001 C CNN
+	1    2250 6500
+	0    1    1    0
+$EndComp
+Wire Wire Line
+	2400 6500 2500 6500
+$Comp
+L device:R R?
+U 1 1 5ADBF4AD
+P 5150 6500
+F 0 "R?" V 4943 6500 50  0000 C CNN
+F 1 "1k" V 5034 6500 50  0000 C CNN
+F 2 "" V 5080 6500 50  0001 C CNN
+F 3 "" H 5150 6500 50  0001 C CNN
+	1    5150 6500
+	0    1    1    0
+$EndComp
+Wire Wire Line
+	5300 6500 5400 6500
 $EndSCHEMATC

Commit message: Finished basic schimatic layout
Parts:
- added C? (x5): 0.33uF, symbol device:C
- added R? (x39): 200, symbol device:R
- gave numbers to parts that had none: 2
Connections:
- net labels added: QH1, QH2, QH3, QH4, RCLK, SER, SRCLK
- wire segments 16 -> 135

Commit message: Annotated schematic
Parts:
- D2: renamed from D?; value LED -> Probe 1
- D3: renamed from D?; value LED -> Probe 2
- D4: renamed from D?; value LED -> Probe 3
- D5: renamed from D?; value LED -> Probe 4
- D6: renamed from D?; value LED -> °C
- D7: renamed from D?; value LED -> °F
- D8: renamed from D?; value LED -> K
- gave numbers to parts that had none: 52
- renumbered U11 to U10, U12 to U11, U13 to U12, U7 to U6, U8 to U7, U9 to U8, U10 to U9

Commit message: Renamed some components
Parts:
- D2: value Probe 1 -> LED Probe 1
- D3: value Probe 2 -> LED Probe 2
- D4: value Probe 3 -> LED Probe 3
- D5: value Probe 4 -> LED Probe 4
- D6: value °C -> LED °C
- D7: value °F -> LED °F
- D8: value K -> LED K
Changed lines of the file:
@@
 P 10550 700
 F 0 "D2" H 10542 445 50  0000 C CNN
-F 1 "Probe 1" H 10542 536 50  0000 C CNN
+F 1 "LED Probe 1" H 10542 536 50  0000 C CNN
 F 2 "" H 10550 700 50  0001 C CNN
 F 3 "~" H 10550 700 50  0001 C CNN
@@
 P 10550 1150
 F 0 "D3" H 10542 895 50  0000 C CNN
-F 1 "Probe 2" H 10542 986 50  0000 C CNN
+F 1 "LED Probe 2" H 10542 986 50  0000 C CNN
 F 2 "" H 10550 1150 50  0001 C CNN
 F 3 "~" H 10550 1150 50  0001 C CNN
@@
 P 10550 1600
 F 0 "D4" H 10542 1345 50  0000 C CNN
-F 1 "Probe 3" H 10542 1436 50  0000 C CNN
+F 1 "LED Probe 3" H 10542 1436 50  0000 C CNN
 F 2 "" H 10550 1600 50  0001 C CNN
 F 3 "~" H 10550 1600 50  0001 C CNN
@@
 P 10550 2100
 F 0 "D5" H 10542 1845 50  0000 C CNN
-F 1 "Probe 4" H 10542 1936 50  0000 C CNN
+F 1 "LED Probe 4" H 10542 1936 50  0000 C CNN
 F 2 "" H 10550 2100 50  0001 C CNN
 F 3 "~" H 10550 2100 50  0001 C CNN
@@
 P 10550 2550
 F 0 "D6" H 10542 2295 50  0000 C CNN
-F 1 "°C" H 10542 2386 50  0000 C CNN
+F 1 "LED °C" H 10542 2386 50  0000 C CNN
 F 2 "" H 10550 2550 50  0001 C CNN
 F 3 "~" H 10550 2550 50  0001 C CNN
@@
 P 10550 3050
 F 0 "D7" H 10542 2795 50  0000 C CNN
-F 1 "°F" H 10542 2886 50  0000 C CNN
+F 1 "LED °F" H 10542 2886 50  0000 C CNN
 F 2 "" H 10550 3050 50  0001 C CNN
 F 3 "~" H 10550 3050 50  0001 C CNN
@@
 P 10550 3550
 F 0 "D8" H 10542 3295 50  0000 C CNN
-F 1 "K" H 10542 3386 50  0000 C CNN
+F 1 "LED K" H 10542 3386 50  0000 C CNN
 F 2 "" H 10550 3550 50  0001 C CNN
 F 3 "~" H 10550 3550 50  0001 C CNN

Commit message: Made footprint for the terminal block
Parts:
- C19, C20, C35, C36, C37, C38, C39: footprint (none) -> Capacitors_SMD:C_0603
- D2, D3, D4, D5, D6, D7, D8: footprint (none) -> LEDs:LED_0603
Changed lines of the file:
@@
 F 0 "D2" H 10542 445 50  0000 C CNN
 F 1 "LED Probe 1" H 10542 536 50  0000 C CNN
-F 2 "" H 10550 700 50  0001 C CNN
+F 2 "LEDs:LED_0603" H 10550 700 50  0001 C CNN
 F 3 "~" H 10550 700 50  0001 C CNN
 	1    10550 700
@@
 F 0 "D3" H 10542 895 50  0000 C CNN
 F 1 "LED Probe 2" H 10542 986 50  0000 C CNN
-F 2 "" H 10550 1150 50  0001 C CNN
+F 2 "LEDs:LED_0603" H 10550 1150 50  0001 C CNN
 F 3 "~" H 10550 1150 50  0001 C CNN
 	1    10550 1150
@@
 F 0 "D4" H 10542 1345 50  0000 C CNN
 F 1 "LED Probe 3" H 10542 1436 50  0000 C CNN
-F 2 "" H 10550 1600 50  0001 C CNN
+F 2 "LEDs:LED_0603" H 10550 1600 50  0001 C CNN
 F 3 "~" H 10550 1600 50  0001 C CNN
 	1    10550 1600
@@
 F 0 "D5" H 10542 1845 50  0000 C CNN
 F 1 "LED Probe 4" H 10542 1936 50  0000 C CNN
-F 2 "" H 10550 2100 50  0001 C CNN
+F 2 "LEDs:LED_0603" H 10550 2100 50  0001 C CNN
 F 3 "~" H 10550 2100 50  0001 C CNN
 	1    10550 2100
@@
 F 0 "D6" H 10542 2295 50  0000 C CNN
 F 1 "LED °C" H 10542 2386 50  0000 C CNN
-F 2 "" H 10550 2550 50  0001 C CNN
+F 2 "LEDs:LED_0603" H 10550 2550 50  0001 C CNN
 F 3 "~" H 10550 2550 50  0001 C CNN
 	1    10550 2550
@@
 F 0 "D7" H 10542 2795 50  0000 C CNN
 F 1 "LED °F" H 10542 2886 50  0000 C CNN
-F 2 "" H 10550 3050 50  0001 C CNN
+F 2 "LEDs:LED_0603" H 10550 3050 50  0001 C CNN
 F 3 "~" H 10550 3050 50  0001 C CNN
 	1    10550 3050
@@
 F 0 "D8" H 10542 3295 50  0000 C CNN
 F 1 "LED K" H 10542 3386 50  0000 C CNN
-F 2 "" H 10550 3550 50  0001 C CNN
+F 2 "LEDs:LED_0603" H 10550 3550 50  0001 C CNN
 F 3 "~" H 10550 3550 50  0001 C CNN
 	1    10550 3550
@@
 F 0 "C19" H 6965 4846 50  0000 L CNN
 F 1 "0.1uF" H 6965 4755 50  0000 L CNN
-F 2 "" H 6888 4650 50  0001 C CNN
+F 2 "Capacitors_SMD:C_0603" H 6888 4650 50  0001 C CNN
 F 3 "" H 6850 4800 50  0001 C CNN
 	1    6850 4800
@@
 F 0 "C20" H 9865 4846 50  0000 L CNN
 F 1 "0.1uF" H 9865 4755 50  0000 L CNN
-F 2 "" H 9788 4650 50  0001 C CNN
+F 2 "Capacitors_SMD:C_0603" H 9788 4650 50  0001 C CNN
 F 3 "" H 9750 4800 50  0001 C CNN
 	1    9750 4800
@@
 F 0 "C37" V 1198 5550 50  0000 C CNN
 F 1 "0.33uF" V 1289 5550 50  0000 C CNN
-F 2 "" H 1488 5400 50  0001 C CNN
+F 2 "Capacitors_SMD:C_0603" H 1488 5400 50  0001 C CNN
 F 3 "" H 1450 5550 50  0001 C CNN
 	1    1450 5550
@@
 F 0 "C38" V 4798 5550 50  0000 C CNN
 F 1 "0.33uF" V 4889 5550 50  0000 C CNN
-F 2 "" H 5088 5400 50  0001 C CNN
+F 2 "Capacitors_SMD:C_0603" H 5088 5400 50  0001 C CNN
 F 3 "" H 5050 5550 50  0001 C CNN
 	1    5050 5550
@@
 F 0 "C36" V 4798 1700 50  0000 C CNN
 F 1 "0.33uF" V 4889 1700 50  0000 C CNN
-F 2 "" H 5088 1550 50  0001 C CNN
+F 2 "Capacitors_SMD:C_0603" H 5088 1550 50  0001 C CNN
 F 3 "" H 5050 1700 50  0001 C CNN
 	1    5050 1700
@@
 F 0 "C35" V 1198 1700 50  0000 C CNN
 F 1 "0.33uF" V 1289 1700 50  0000 C CNN
-F 2 "" H 1488 1550 50  0001 C CNN
+F 2 "Capacitors_SMD:C_0603" H 1488 1550 50  0001 C CNN
 F 3 "" H 1450 1700 50  0001 C CNN
 	1    1450 1700
@@
 F 0 "C39" V 8448 1200 50  0000 C CNN
 F 1 "0.33uF" V 8539 1200 50  0000 C CNN
-F 2 "" H 8738 1050 50  0001 C CNN
+F 2 "Capacitors_SMD:C_0603" H 8738 1050 50  0001 C CNN
 F 3 "" H 8700 1200 50  0001 C CNN
 	1    8700 1200

Commit message: Added the components and generaterd the netlist
Parts:
- R11, R12, R13, R14, R15, R16, R17, R18, R19, R20, R21, R22, R23, R24, R25, R26, R27, R28, R29, R30, R31, R32, R33, R34, R35, R36, R37, R38, R39, R40, R41, R42, R43, R44, R45, R46, R47, R48, R49: footprint (none) -> Resistors_SMD:R_0805
- R50, R51, R55, R56: footprint (none) -> Resistors_SMD:R_0402
- SW3, SW4: footprint (none) -> Buttons_Switches_SMD:SW_SPST_PTS645
- U10, U6, U7, U8, U9: footprint (none) -> Housings_SSOP:TSSOP-16_4.4x5mm_Pitch0.65mm

Commit message: Started pcb design
Parts:
- U11, U12: footprint Displays_7-Segment:HDSP-521E -> Display:HDSP-521E
Changed lines of the file:
@@
 F 0 "U12" H 3400 7017 50  0000 C CNN
 F 1 "HDSP-521E-Display" H 3400 6926 50  0000 C CNN
-F 2 "Displays_7-Segment:HDSP-521E" H 3420 5700 50  0001 C CNN
+F 2 "Display:HDSP-521E" H 3420 5700 50  0001 C CNN
 F 3 "" H 3280 6450 50  0001 C CNN
 	1    3400 6450
@@
 F 0 "U11" H 3400 3167 50  0000 C CNN
 F 1 "HDSP-521E-Display" H 3400 3076 50  0000 C CNN
-F 2 "Displays_7-Segment:HDSP-521E" H 3420 1850 50  0001 C CNN
+F 2 "Display:HDSP-521E" H 3420 1850 50  0001 C CNN
 F 3 "" H 3280 2600 50  0001 C CNN
 	1    3400 2600
