File: Thermocouple-Data-Logger/Display.sch (KiCad schematic (older format))
At the start: 66 parts, among them SW3 Select/Calibrate, SW4 Cycle/Menu, U10 74HC595, U11 HDSP-521E-Display, U12 HDSP-521E-Display, U6 74HC595, U7 74HC595, U8 74HC595, U9 74HC595

Commit message: Changed capacitor values and component layout
Parts:
- C19, C20: footprint Capacitors_SMD:C_0603 -> Capacitors_SMD:C_0402
- C35, C36, C37, C38, C39: value 0.33uF -> 0.1uF; footprint Capacitors_SMD:C_0603 -> Capacitors_SMD:C_0402
Changed lines of the file:
@@
 F 0 "C19" H 6965 4846 50  0000 L CNN
 F 1 "0.1uF" H 6965 4755 50  0000 L CNN
-F 2 "Capacitors_SMD:C_0603" H 6888 4650 50  0001 C CNN
+F 2 "Capacitors_SMD:C_0402" H 6888 4650 50  0001 C CNN
 F 3 "" H 6850 4800 50  0001 C CNN
 	1    6850 4800
@@
 F 0 "C20" H 9865 4846 50  0000 L CNN
 F 1 "0.1uF" H 9865 4755 50  0000 L CNN
-F 2 "Capacitors_SMD:C_0603" H 9788 4650 50  0001 C CNN
+F 2 "Capacitors_SMD:C_0402" H 9788 4650 50  0001 C CNN
 F 3 "" H 9750 4800 50  0001 C CNN
 	1    9750 4800
@@
 P 1450 5550
 F 0 "C37" V 1198 5550 50  0000 C CNN
-F 1 "0.33uF" V 1289 5550 50  0000 C CNN
-F 2 "Capacitors_SMD:C_0603" H 1488 5400 50  0001 C CNN
+F 1 "0.1uF" V 1289 5550 50  0000 C CNN
+F 2 "Capacitors_SMD:C_0402" H 1488 5400 50  0001 C CNN
 F 3 "" H 1450 5550 50  0001 C CNN
 	1    1450 5550
@@
 P 5050 5550
 F 0 "C38" V 4798 5550 50  0000 C CNN
-F 1 "0.33uF" V 4889 5550 50  0000 C CNN
-F 2 "Capacitors_SMD:C_0603" H 5088 5400 50  0001 C CNN
+F 1 "0.1uF" V 4889 5550 50  0000 C CNN
+F 2 "Capacitors_SMD:C_0402" H 5088 5400 50  0001 C CNN
 F 3 "" H 5050 5550 50  0001 C CNN
 	1    5050 5550
@@
 P 5050 1700
 F 0 "C36" V 4798 1700 50  0000 C CNN
-F 1 "0.33uF" V 4889 1700 50  0000 C CNN
-F 2 "Capacitors_SMD:C_0603" H 5088 1550 50  0001 C CNN
+F 1 "0.1uF" V 4889 1700 50  0000 C CNN
+F 2 "Capacitors_SMD:C_0402" H 5088 1550 50  0001 C CNN
 F 3 "" H 5050 1700 50  0001 C CNN
 	1    5050 1700
@@
 P 1450 1700
 F 0 "C35" V 1198 1700 50  0000 C CNN
-F 1 "0.33uF" V 1289 1700 50  0000 C CNN
-F 2 "Capacitors_SMD:C_0603" H 1488 1550 50  0001 C CNN
+F 1 "0.1uF" V 1289 1700 50  0000 C CNN
+F 2 "Capacitors_SMD:C_0402" H 1488 1550 50  0001 C CNN
 F 3 "" H 1450 1700 50  0001 C CNN
 	1    1450 1700
@@
 P 8700 1200
 F 0 "C39" V 8448 1200 50  0000 C CNN
-F 1 "0.33uF" V 8539 1200 50  0000 C CNN
-F 2 "Capacitors_SMD:C_0603" H 8738 1050 50  0001 C CNN
+F 1 "0.1uF" V 8539 1200 50  0000 C CNN
+F 2 "Capacitors_SMD:C_0402" H 8738 1050 50  0001 C CNN
 F 3 "" H 8700 1200 50  0001 C CNN
 	1    8700 1200

Commit message: Started laying down traces
Changed lines of the file:
@@
 Text HLabel 5700 2800 2    50   Input ~ 0
 RCLK
-Text HLabel 1050 6350 0    50   Input ~ 0
+Text HLabel 1100 6350 0    50   Input ~ 0
 SRCLK
 Text HLabel 1100 6650 0    50   Input ~ 0

Commit message: Changed the microcontroller from qfn to tqfp
Parts:
- C19, C20, C35, C36, C37, C38, C39: symbol device:C -> Thermocouple-Data-Logger-rescue:C-device
- D2, D3, D4, D5, D6, D7, D8: symbol device:LED -> Thermocouple-Data-Logger-rescue:LED-device
- R11, R12, R13, R14, R15, R16, R17, R18, R19, R20, R21, R22, R23, R24, R25, R26, R27, R28, R29, R30, R31, R32, R33, R34, R35, R36, R37, R38, R39, R40, R41, R42, R43, R44, R45, R46, R47, R48, R49, R50, R51, R55, R56: symbol device:R -> Thermocouple-Data-Logger-rescue:R-device
- U10, U6, U7, U8, U9: symbol Logic_74xx:74HC595 -> Thermocouple-Data-Logger-rescue:74HC595-Logic_74xx
Changed lines of the file:
@@
 $EndDescr
 $Comp
-L Logic_74xx:74HC595 U6
+L Thermocouple-Data-Logger-rescue:74HC595-Logic_74xx U6
 U 1 1 5A86784D
 P 1600 2700
@@
 $EndComp
 $Comp
-L Logic_74xx:74HC595 U8
+L Thermocouple-Data-Logger-rescue:74HC595-Logic_74xx U8
 U 1 1 5A86785B
 P 1600 6550
@@
 $EndComp
 $Comp
-L Logic_74xx:74HC595 U9
+L Thermocouple-Data-Logger-rescue:74HC595-Logic_74xx U9
 U 1 1 5A867862
 P 5200 6550
@@
 VCC
 $Comp
-L Logic_74xx:74HC595 U10
+L Thermocouple-Data-Logger-rescue:74HC595-Logic_74xx U10
 U 1 1 5A868ED4
 P 8850 2200
@@
 $EndComp
 $Comp
-L device:LED D2
+L Thermocouple-Data-Logger-rescue:LED-device D2
 U 1 1 5A8DC5E4
 P 10550 700
@@
 $EndComp
 $Comp
-L device:LED D3
+L Thermocouple-Data-Logger-rescue:LED-device D3
 U 1 1 5A8DC6B4
 P 10550 1150
@@
 $EndComp
 $Comp
-L device:LED D4
+L Thermocouple-Data-Logger-rescue:LED-device D4
 U 1 1 5A8DC6DB
 P 10550 1600
@@
 $EndComp
 $Comp
-L device:LED D5
+L Thermocouple-Data-Logger-rescue:LED-device D5
 U 1 1 5A8DC706
 P 10550 2100
@@
 $EndComp
 $Comp
-L device:LED D6
+L Thermocouple-Data-Logger-rescue:LED-device D6
 U 1 1 5A8DC734
 P 10550 2550
@@
 $EndComp
 $Comp
-L device:LED D7
+L Thermocouple-Data-Logger-rescue:LED-device D7
 U 1 1 5A8DC77F
 P 10550 3050
@@
 $EndComp
 $Comp
-L device:LED D8
+L Thermocouple-Data-Logger-rescue:LED-device D8
 U 1 1 5A8DC7B7
 P 10550 3550
@@
 	7850 5150 8000 5150
 $Comp
-L device:R R55
+L Thermocouple-Data-Logger-rescue:R-device R55
 U 1 1 5AD8AEEC
 P 6850 5450
@@
 	10750 5150 10900 5150
 $Comp
-L device:R R56
+L Thermocouple-Data-Logger-rescue:R-device R56
 U 1 1 5AD8C3A0
 P 9750 5450
@@
 	6850 5150 7050 5150
 $Comp
-L device:C C19
+L Thermocouple-Data-Logger-rescue:C-device C19
 U 1 1 5ADBEA6C
 P 6850 4800
@@
 $EndComp
 $Comp
-L device:C C20
+L Thermocouple-Data-Logger-rescue:C-device C20
 U 1 1 5ADBECAE
 P 9750 4800
@@
 	6850 4650 6850 4450
 $Comp
-L device:R R50
+L Thermocouple-Data-Logger-rescue:R-device R50
 U 1 1 5ADBF30B
 P 7200 5150
@@
 	7350 5150 7450 5150
 $Comp
-L device:R R51
+L Thermocouple-Data-Logger-rescue:R-device R51
 U 1 1 5ADBF4AD
 P 10100 5150
@@
 	950  2900 1100 2900
 $Comp
-L device:R R27
+L Thermocouple-Data-Logger-rescue:R-device R27
 U 1 1 5AA2E7D1
 P 2450 6150
@@
 	2100 6250 2300 6250
 $Comp
-L device:R R28
+L Thermocouple-Data-Logger-rescue:R-device R28
 U 1 1 5AA309AA
 P 2450 6250
@@
 	2100 6350 2300 6350
 $Comp
-L device:R R29
+L Thermocouple-Data-Logger-rescue:R-device R29
 U 1 1 5AA322B2
 P 2450 6350
@@
 	2100 6450 2300 6450
 $Comp
-L device:R R30
+L Thermocouple-Data-Logger-rescue:R-device R30
 U 1 1 5AA33DF0
 P 2450 6450
@@
 	2100 6550 2300 6550
 $Comp
-L device:R R31
+L Thermocouple-Data-Logger-rescue:R-device R31
 U 1 1 5AA35B73
 P 2450 6550
@@
 	2100 6650 2300 6650
 $Comp
-L device:R R32
+L Thermocouple-Data-Logger-rescue:R-device R32
 U 1 1 5AA37B4A
 P 2450 6650
@@
 	2100 6750 2300 6750
 $Comp
-L device:R R33
+L Thermocouple-Data-Logger-rescue:R-device R33
 U 1 1 5AA39D84
 P 2450 6750
@@
 	2100 6850 2300 6850
 $Comp
-L device:R R34
+L Thermocouple-Data-Logger-rescue:R-device R34
 U 1 1 5AA3C232
 P 2450 6850
@@
 	2600 6850 2800 6850
 $Comp
-L device:R R35
+L Thermocouple-Data-Logger-rescue:R-device R35
 U 1 1 5AA41188
 P 4350 6150
@@
 	4500 6150 4700 6150
 $Comp
-L device:R R36
+L Thermocouple-Data-Logger-rescue:R-device R36
 U 1 1 5AA43AC2
 P 4350 6250
@@
 	4500 6250 4700 6250
 $Comp
-L device:R R37
+L Thermocouple-Data-Logger-rescue:R-device R37
 U 1 1 5AA4650C
 P 4350 6350
@@
 	4500 6350 4700 6350
 $Comp
-L device:R R38
+L Thermocouple-Data-Logger-rescue:R-device R38
 U 1 1 5AA49064
 P 4350 6450
@@
 	4500 6450 4700 6450
 $Comp
-L device:R R39
+L Thermocouple-Data-Logger-rescue:R-device R39
 U 1 1 5AA4BCC7
 P 4350 6550
@@
 	4500 6550 4700 6550
 $Comp
-L device:R R40
+L Thermocouple-Data-Logger-rescue:R-device R40
 U 1 1 5AA4EA2F
 P 4350 6650
@@
 	4500 6650 4700 6650
 $Comp
-L device:R R41
+L Thermocouple-Data-Logger-rescue:R-device R41
 U 1 1 5AA518A1
 P 4350 6750
@@
 	4500 6750 4700 6750
 $Comp
-L device:R R42
+L Thermocouple-Data-Logger-rescue:R-device R42
 U 1 1 5AA54817
 P 4350 6850
@@
 	9350 700  10000 700
 $Comp
-L device:R R43
+L Thermocouple-Data-Logger-rescue:R-device R43
 U 1 1 5AA5AAF6
 P 10150 700
@@
 	10300 700  10400 700
 $Comp
-L device:R R44
+L Thermocouple-Data-Logger-rescue:R-device R44
 U 1 1 5AA5AB84
 P 10150 1150
@@
 	10300 1150 10400 1150
 $Comp
-L device:R R45
+L Thermocouple-Data-Logger-rescue:R-device R45
 U 1 1 5AA66F34
 P 10150 1600
@@
 	10300 1600 10400 1600
 $Comp
-L device:R R46
+L Thermocouple-Data-Logger-rescue:R-device R46
 U 1 1 5AA66FA5
 P 10150 2100
@@
 	10300 2100 10400 2100
 $Comp
-L device:R R47
+L Thermocouple-Data-Logger-rescue:R-device R47
 U 1 1 5AA67015
 P 10150 2550
@@
 	10300 2550 10400 2550
 $Comp
-L device:R R48
+L Thermocouple-Data-Logger-rescue:R-device R48
 U 1 1 5AA67088
 P 10150 3050
@@
 	10300 3050 10400 3050
 $Comp
-L device:R R49
+L Thermocouple-Data-Logger-rescue:R-device R49
 U 1 1 5AA670FC
 P 10150 3550
@@
 	10300 3550 10400 3550
 $Comp
-L Logic_74xx:74HC595 U7
+L Thermocouple-Data-Logger-rescue:74HC595-Logic_74xx U7
 U 1 1 5A867854
 P 5200 2700
@@
 $EndComp
 $Comp
-L device:R R19
+L Thermocouple-Data-Logger-rescue:R-device R19
 U 1 1 5AA8C43B
 P 4350 2300
@@
 	4500 2300 4700 2300
 $Comp
-L device:R R20
+L Thermocouple-Data-Logger-rescue:R-device R20
 U 1 1 5AA9141C
 P 4350 2400
@@
 	4500 2400 4700 2400
 $Comp
-L device:R R21
+L Thermocouple-Data-Logger-rescue:R-device R21
 U 1 1 5AA93E63
 P 4350 2500
@@
 	4500 2500 4700 2500
 $Comp
-L device:R R22
+L Thermocouple-Data-Logger-rescue:R-device R22
 U 1 1 5AA96B27
 P 4350 2600
@@
 	4500 2600 4700 2600
 $Comp
-L device:R R23
+L Thermocouple-Data-Logger-rescue:R-device R23
 U 1 1 5AA99A77
 P 4350 2700
@@
 	4500 2700 4700 2700
 $Comp
-L device:R R24
+L Thermocouple-Data-Logger-rescue:R-device R24
 U 1 1 5AA9CC62
 P 4350 2800
@@
 	4500 2800 4700 2800
 $Comp
-L device:R R25
+L Thermocouple-Data-Logger-rescue:R-device R25
 U 1 1 5AAA00F8
 P 4350 2900
@@
 	4500 2900 4700 2900
 $Comp
-L device:R R26
+L Thermocouple-Data-Logger-rescue:R-device R26
 U 1 1 5AAA3846
 P 4350 3000
@@
 	4500 3000 4700 3000
 $Comp
-L device:R R11
+L Thermocouple-Data-Logger-rescue:R-device R11
 U 1 1 5AAA74B3
 P 2450 2300
@@
 	2100 2300 2300 2300
 $Comp
-L device:R R12
+L Thermocouple-Data-Logger-rescue:R-device R12
 U 1 1 5AAAF076
 P 2450 2400
@@
 	2100 2400 2300 2400
 $Comp
-L device:R R13
+L Thermocouple-Data-Logger-rescue:R-device R13
 U 1 1 5AAB31BC
 P 2450 2500
@@
 	2100 2500 2300 2500
 $Comp
-L device:R R14
+L Thermocouple-Data-Logger-rescue:R-device R14
 U 1 1 5AAB76B2
 P 2450 2600
@@
 	2100 2600 2300 2600
 $Comp
-L device:R R15
+L Thermocouple-Data-Logger-rescue:R-device R15
 U 1 1 5AABBF66
 P 2450 2700
@@
 	2100 2700 2300 2700
 $Comp
-L device:R R16
+L Thermocouple-Data-Logger-rescue:R-device R16
 U 1 1 5AAC0BE9
 P 2450 2800
@@
 	2100 2800 2300 2800
 $Comp
-L device:R R17
+L Thermocouple-Data-Logger-rescue:R-device R17
 U 1 1 5AAC5C48
 P 2450 2900
@@
 	2100 2900 2300 2900
 $Comp
-L device:R R18
+L Thermocouple-Data-Logger-rescue:R-device R18
 U 1 1 5AACB091
 P 2450 3000
@@
 $EndComp
 $Comp
-L device:C C37
+L Thermocouple-Data-Logger-rescue:C-device C37
 U 1 1 5AB08FD8
 P 1450 5550
@@
 VCC
 $Comp
-L device:C C38
+L Thermocouple-Data-Logger-rescue:C-device C38
 U 1 1 5AB149FA
 P 5050 5550
@@
 VCC
 $Comp
-L device:C C36
+L Thermocouple-Data-Logger-rescue:C-device C36
 U 1 1 5AB1A8E3
 P 5050 1700
@@
 VCC
 $Comp
-L device:C C35
+L Thermocouple-Data-Logger-rescue:C-device C35
 U 1 1 5AB207BE
 P 1450 1700
@@
 VCC
 $Comp
-L device:C C39
+L Thermocouple-Data-Logger-rescue:C-device C39
 U 1 1 5AB268F4
 P 8700 1200
