File: Thermocouple-Data-Logger/Thermocouple.sch (KiCad schematic (older format))
At the start: 6 parts

Commit message: Added a lot more to the schimatic
Parts:
- added C? (x4): 0.1uF, symbol device:C
- added C? (x8): 0.01uF, symbol device:C
- added C? (x6): 0.33uF, symbol device:C
- added J? (x3): Conn_01x02, symbol Connector:Conn_01x02
- added R? (x6): 100, symbol device:R
- added U? (x3): MAX31856, Housings_SSOP:TSSOP-14_4.4x5mm_Pitch0.65mm, symbol sensors:MAX31856
Connections:
- net labels added: CS1, CS2, CS3, CS4, DRDY1, DRDY2, DRDY3, DRDY4, FAULT1, FAULT2, FAULT3, FAULT4, SCK, SDI, SDO, VCC2, VCC3, VCC4
- wire segments 23 -> 128

Commit message: Added switches
Parts:
- gave numbers to parts that had none: 4
Changed lines of the file:
@@
 $EndDescr
 $Comp
-L sensors:MAX31856 U?
+L sensors:MAX31856 U3
 U 1 1 5A878CB3
 P 2900 2450
-F 0 "U?" H 2900 3228 50  0000 C CNN
+F 0 "U3" H 2900 3228 50  0000 C CNN
 F 1 "MAX31856" H 2900 3137 50  0000 C CNN
 F 2 "Housings_SSOP:TSSOP-14_4.4x5mm_Pitch0.65mm" H 3050 1900 50  0001 L CNN
@@
 SDI
 $Comp
-L sensors:MAX31856 U?
+L sensors:MAX31856 U5
 U 1 1 5A96C92D
 P 2950 5150
-F 0 "U?" H 2950 5928 50  0000 C CNN
+F 0 "U5" H 2950 5928 50  0000 C CNN
 F 1 "MAX31856" H 2950 5837 50  0000 C CNN
 F 2 "Housings_SSOP:TSSOP-14_4.4x5mm_Pitch0.65mm" H 3100 4600 50  0001 L CNN
@@
 SDI
 $Comp
-L sensors:MAX31856 U?
+L sensors:MAX31856 U4
 U 1 1 5A96DCFD
 P 6900 2450
-F 0 "U?" H 6900 3228 50  0000 C CNN
+F 0 "U4" H 6900 3228 50  0000 C CNN
 F 1 "MAX31856" H 6900 3137 50  0000 C CNN
 F 2 "Housings_SSOP:TSSOP-14_4.4x5mm_Pitch0.65mm" H 7050 1900 50  0001 L CNN
@@
 SDI
 $Comp
-L sensors:MAX31856 U?
+L sensors:MAX31856 U6
 U 1 1 5A9701A9
 P 7000 5150
-F 0 "U?" H 7000 5928 50  0000 C CNN
+F 0 "U6" H 7000 5928 50  0000 C CNN
 F 1 "MAX31856" H 7000 5837 50  0000 C CNN
 F 2 "Housings_SSOP:TSSOP-14_4.4x5mm_Pitch0.65mm" H 7150 4600 50  0001 L CNN

Commit message: Annotated schematic
Parts:
- gave numbers to parts that had none: 32
- renumbered U3 to U2, U4 to U3, U5 to U4, U6 to U5

Commit message: Renamed some components
Parts:
- J2: value Conn_01x02 -> Probe 1
- J3: value Conn_01x02 -> Probe 2
- J4: value Conn_01x02 -> Probe 3
- J5: value Conn_01x02 -> Probe 4
Changed lines of the file:
@@
 P 1000 2450
 F 0 "J2" H 920 2125 50  0000 C CNN
-F 1 "Conn_01x02" H 920 2216 50  0000 C CNN
+F 1 "Probe 1" H 920 2216 50  0000 C CNN
 F 2 "" H 1000 2450 50  0001 C CNN
 F 3 "~" H 1000 2450 50  0001 C CNN
@@
 P 1050 5150
 F 0 "J4" H 970 4825 50  0000 C CNN
-F 1 "Conn_01x02" H 970 4916 50  0000 C CNN
+F 1 "Probe 3" H 970 4916 50  0000 C CNN
 F 2 "" H 1050 5150 50  0001 C CNN
 F 3 "~" H 1050 5150 50  0001 C CNN
@@
 P 5000 2450
 F 0 "J3" H 4920 2125 50  0000 C CNN
-F 1 "Conn_01x02" H 4920 2216 50  0000 C CNN
+F 1 "Probe 2" H 4920 2216 50  0000 C CNN
 F 2 "" H 5000 2450 50  0001 C CNN
 F 3 "~" H 5000 2450 50  0001 C CNN
@@
 P 5100 5150
 F 0 "J5" H 5020 4825 50  0000 C CNN
-F 1 "Conn_01x02" H 5020 4916 50  0000 C CNN
+F 1 "Probe 4" H 5020 4916 50  0000 C CNN
 F 2 "" H 5100 5150 50  0001 C CNN
 F 3 "~" H 5100 5150 50  0001 C CNN

Commit message: Made footprint for the terminal block
Parts:
- C10, C11, C4, C5, C6, C7, C8, C9: footprint (none) -> Capacitors_SMD:C_0402
- C15, C16, C17, C18, C25, C26, C27, C28, C29, C30, C31, C32: footprint (none) -> Capacitors_SMD:C_0603
- J2, J3, J4, J5: footprint (none) -> TerminalBlock-PTSA:TeaminalBlock_Phonix_PTSA-3.5mm_2pol
Changed lines of the file:
@@
 F 0 "J2" H 920 2125 50  0000 C CNN
 F 1 "Probe 1" H 920 2216 50  0000 C CNN
-F 2 "" H 1000 2450 50  0001 C CNN
+F 2 "TerminalBlock-PTSA:TeaminalBlock_Phonix_PTSA-3.5mm_2pol" H 1000 2450 50  0001 C CNN
 F 3 "~" H 1000 2450 50  0001 C CNN
 	1    1000 2450
@@
 F 0 "C26" H 3665 1346 50  0000 L CNN
 F 1 "0.33uF" H 3665 1255 50  0000 L CNN
-F 2 "" H 3588 1150 50  0001 C CNN
+F 2 "Capacitors_SMD:C_0603" H 3588 1150 50  0001 C CNN
 F 3 "" H 3550 1300 50  0001 C CNN
 	1    3550 1300
@@
 F 0 "C25" H 2365 1346 50  0000 L CNN
 F 1 "0.33uF" H 2365 1255 50  0000 L CNN
-F 2 "" H 2288 1150 50  0001 C CNN
+F 2 "Capacitors_SMD:C_0603" H 2288 1150 50  0001 C CNN
 F 3 "" H 2250 1300 50  0001 C CNN
 	1    2250 1300
@@
 F 0 "C15" H 1965 2446 50  0000 L CNN
 F 1 "0.1uF" H 1965 2355 50  0000 L CNN
-F 2 "" H 1888 2250 50  0001 C CNN
+F 2 "Capacitors_SMD:C_0603" H 1888 2250 50  0001 C CNN
 F 3 "" H 1850 2400 50  0001 C CNN
 	1    1850 2400
@@
 F 0 "C5" H 1965 2996 50  0000 L CNN
 F 1 "0.01uF" H 1965 2905 50  0000 L CNN
-F 2 "" H 1888 2800 50  0001 C CNN
+F 2 "Capacitors_SMD:C_0402" H 1888 2800 50  0001 C CNN
 F 3 "" H 1850 2950 50  0001 C CNN
 	1    1850 2950
@@
 F 0 "C4" H 1965 1896 50  0000 L CNN
 F 1 "0.01uF" H 1965 1805 50  0000 L CNN
-F 2 "" H 1888 1700 50  0001 C CNN
+F 2 "Capacitors_SMD:C_0402" H 1888 1700 50  0001 C CNN
 F 3 "" H 1850 1850 50  0001 C CNN
 	1    1850 1850
@@
 F 0 "J4" H 970 4825 50  0000 C CNN
 F 1 "Probe 3" H 970 4916 50  0000 C CNN
-F 2 "" H 1050 5150 50  0001 C CNN
+F 2 "TerminalBlock-PTSA:TeaminalBlock_Phonix_PTSA-3.5mm_2pol" H 1050 5150 50  0001 C CNN
 F 3 "~" H 1050 5150 50  0001 C CNN
 	1    1050 5150
@@
 F 0 "C30" H 3715 4046 50  0000 L CNN
 F 1 "0.33uF" H 3715 3955 50  0000 L CNN
-F 2 "" H 3638 3850 50  0001 C CNN
+F 2 "Capacitors_SMD:C_0603" H 3638 3850 50  0001 C CNN
 F 3 "" H 3600 4000 50  0001 C CNN
 	1    3600 4000
@@
 F 0 "C29" H 2415 4046 50  0000 L CNN
 F 1 "0.33uF" H 2415 3955 50  0000 L CNN
-F 2 "" H 2338 3850 50  0001 C CNN
+F 2 "Capacitors_SMD:C_0603" H 2338 3850 50  0001 C CNN
 F 3 "" H 2300 4000 50  0001 C CNN
 	1    2300 4000
@@
 F 0 "C17" H 2015 5146 50  0000 L CNN
 F 1 "0.1uF" H 2015 5055 50  0000 L CNN
-F 2 "" H 1938 4950 50  0001 C CNN
+F 2 "Capacitors_SMD:C_0603" H 1938 4950 50  0001 C CNN
 F 3 "" H 1900 5100 50  0001 C CNN
 	1    1900 5100
@@
 F 0 "C9" H 2015 5696 50  0000 L CNN
 F 1 "0.01uF" H 2015 5605 50  0000 L CNN
-F 2 "" H 1938 5500 50  0001 C CNN
+F 2 "Capacitors_SMD:C_0402" H 1938 5500 50  0001 C CNN
 F 3 "" H 1900 5650 50  0001 C CNN
 	1    1900 5650
@@
 F 0 "C8" H 2015 4596 50  0000 L CNN
 F 1 "0.01uF" H 2015 4505 50  0000 L CNN
-F 2 "" H 1938 4400 50  0001 C CNN
+F 2 "Capacitors_SMD:C_0402" H 1938 4400 50  0001 C CNN
 F 3 "" H 1900 4550 50  0001 C CNN
 	1    1900 4550
@@
 F 0 "J3" H 4920 2125 50  0000 C CNN
 F 1 "Probe 2" H 4920 2216 50  0000 C CNN
-F 2 "" H 5000 2450 50  0001 C CNN
+F 2 "TerminalBlock-PTSA:TeaminalBlock_Phonix_PTSA-3.5mm_2pol" H 5000 2450 50  0001 C CNN
 F 3 "~" H 5000 2450 50  0001 C CNN
 	1    5000 2450
@@
 F 0 "C28" H 7665 1346 50  0000 L CNN
 F 1 "0.33uF" H 7665 1255 50  0000 L CNN
-F 2 "" H 7588 1150 50  0001 C CNN
+F 2 "Capacitors_SMD:C_0603" H 7588 1150 50  0001 C CNN
 F 3 "" H 7550 1300 50  0001 C CNN
 	1    7550 1300
@@
 F 0 "C27" H 6365 1346 50  0000 L CNN
 F 1 "0.33uF" H 6365 1255 50  0000 L CNN
-F 2 "" H 6288 1150 50  0001 C CNN
+F 2 "Capacitors_SMD:C_0603" H 6288 1150 50  0001 C CNN
 F 3 "" H 6250 1300 50  0001 C CNN
 	1    6250 1300
@@
 F 0 "C16" H 5965 2446 50  0000 L CNN
 F 1 "0.1uF" H 5965 2355 50  0000 L CNN
-F 2 "" H 5888 2250 50  0001 C CNN
+F 2 "Capacitors_SMD:C_0603" H 5888 2250 50  0001 C CNN
 F 3 "" H 5850 2400 50  0001 C CNN
 	1    5850 2400
@@
 F 0 "C7" H 5965 2996 50  0000 L CNN
 F 1 "0.01uF" H 5965 2905 50  0000 L CNN
-F 2 "" H 5888 2800 50  0001 C CNN
+F 2 "Capacitors_SMD:C_0402" H 5888 2800 50  0001 C CNN
 F 3 "" H 5850 2950 50  0001 C CNN
 	1    5850 2950
@@
 F 0 "C6" H 5965 1896 50  0000 L CNN
 F 1 "0.01uF" H 5965 1805 50  0000 L CNN
-F 2 "" H 5888 1700 50  0001 C CNN
+F 2 "Capacitors_SMD:C_0402" H 5888 1700 50  0001 C CNN
 F 3 "" H 5850 1850 50  0001 C CNN
 	1    5850 1850
@@
 F 0 "J5" H 5020 4825 50  0000 C CNN
 F 1 "Probe 4" H 5020 4916 50  0000 C CNN
-F 2 "" H 5100 5150 50  0001 C CNN
+F 2 "TerminalBlock-PTSA:TeaminalBlock_Phonix_PTSA-3.5mm_2pol" H 5100 5150 50  0001 C CNN
 F 3 "~" H 5100 5150 50  0001 C CNN
 	1    5100 5150
@@
 F 0 "C32" H 7765 4046 50  0000 L CNN
 F 1 "0.33uF" H 7765 3955 50  0000 L CNN
-F 2 "" H 7688 3850 50  0001 C CNN
+F 2 "Capacitors_SMD:C_0603" H 7688 3850 50  0001 C CNN
 F 3 "" H 7650 4000 50  0001 C CNN
 	1    7650 4000
@@
 F 0 "C31" H 6465 4046 50  0000 L CNN
 F 1 "0.33uF" H 6465 3955 50  0000 L CNN
-F 2 "" H 6388 3850 50  0001 C CNN
+F 2 "Capacitors_SMD:C_0603" H 6388 3850 50  0001 C CNN
 F 3 "" H 6350 4000 50  0001 C CNN
 	1    6350 4000
@@
 F 0 "C18" H 6065 5146 50  0000 L CNN
 F 1 "0.1uF" H 6065 5055 50  0000 L CNN
-F 2 "" H 5988 4950 50  0001 C CNN
+F 2 "Capacitors_SMD:C_0603" H 5988 4950 50  0001 C CNN
 F 3 "" H 5950 5100 50  0001 C CNN
 	1    5950 5100
@@
 F 0 "C11" H 6065 5696 50  0000 L CNN
 F 1 "0.01uF" H 6065 5605 50  0000 L CNN
-F 2 "" H 5988 5500 50  0001 C CNN
+F 2 "Capacitors_SMD:C_0402" H 5988 5500 50  0001 C CNN
 F 3 "" H 5950 5650 50  0001 C CNN
 	1    5950 5650
@@
 F 0 "C10" H 6065 4596 50  0000 L CNN
 F 1 "0.01uF" H 6065 4505 50  0000 L CNN
-F 2 "" H 5988 4400 50  0001 C CNN
+F 2 "Capacitors_SMD:C_0402" H 5988 4400 50  0001 C CNN
 F 3 "" H 5950 4550 50  0001 C CNN
 	1    5950 4550

Commit message: Added the components and generaterd the netlist
Parts:
- R0, R1, R2, R3, R4, R5, R6, R7: footprint (none) -> Resistors_SMD:R_0603
Changed lines of the file:
@@
 F 0 "R0" V 1293 2000 50  0000 C CNN
 F 1 "100" V 1384 2000 50  0000 C CNN
-F 2 "" V 1430 2000 50  0001 C CNN
+F 2 "Resistors_SMD:R_0603" V 1430 2000 50  0001 C CNN
 F 3 "" H 1500 2000 50  0001 C CNN
 	1    1500 2000
@@
 F 0 "R1" V 1293 2800 50  0000 C CNN
 F 1 "100" V 1384 2800 50  0000 C CNN
-F 2 "" V 1430 2800 50  0001 C CNN
+F 2 "Resistors_SMD:R_0603" V 1430 2800 50  0001 C CNN
 F 3 "" H 1500 2800 50  0001 C CNN
 	1    1500 2800
@@
 F 0 "R4" V 1343 4700 50  0000 C CNN
 F 1 "100" V 1434 4700 50  0000 C CNN
-F 2 "" V 1480 4700 50  0001 C CNN
+F 2 "Resistors_SMD:R_0603" V 1480 4700 50  0001 C CNN
 F 3 "" H 1550 4700 50  0001 C CNN
 	1    1550 4700
@@
 F 0 "R5" V 1343 5500 50  0000 C CNN
 F 1 "100" V 1434 5500 50  0000 C CNN
-F 2 "" V 1480 5500 50  0001 C CNN
+F 2 "Resistors_SMD:R_0603" V 1480 5500 50  0001 C CNN
 F 3 "" H 1550 5500 50  0001 C CNN
 	1    1550 5500
@@
 F 0 "R2" V 5293 2000 50  0000 C CNN
 F 1 "100" V 5384 2000 50  0000 C CNN
-F 2 "" V 5430 2000 50  0001 C CNN
+F 2 "Resistors_SMD:R_0603" V 5430 2000 50  0001 C CNN
 F 3 "" H 5500 2000 50  0001 C CNN
 	1    5500 2000
@@
 F 0 "R3" V 5293 2800 50  0000 C CNN
 F 1 "100" V 5384 2800 50  0000 C CNN
-F 2 "" V 5430 2800 50  0001 C CNN
+F 2 "Resistors_SMD:R_0603" V 5430 2800 50  0001 C CNN
 F 3 "" H 5500 2800 50  0001 C CNN
 	1    5500 2800
@@
 F 0 "R6" V 5393 4700 50  0000 C CNN
 F 1 "100" V 5484 4700 50  0000 C CNN
-F 2 "" V 5530 4700 50  0001 C CNN
+F 2 "Resistors_SMD:R_0603" V 5530 4700 50  0001 C CNN
 F 3 "" H 5600 4700 50  0001 C CNN
 	1    5600 4700
@@
 F 0 "R7" V 5393 5500 50  0000 C CNN
 F 1 "100" V 5484 5500 50  0000 C CNN
-F 2 "" V 5530 5500 50  0001 C CNN
+F 2 "Resistors_SMD:R_0603" V 5530 5500 50  0001 C CNN
 F 3 "" H 5600 5500 50  0001 C CNN
 	1    5600 5500
