File: Thermocouple-Data-Logger/Thermocouple.sch (KiCad schematic (older format))
At the start: 36 parts, among them J2 Probe 1, J3 Probe 2, J4 Probe 3, J5 Probe 4, U2 MAX31856, U3 MAX31856, U4 MAX31856, U5 MAX31856

Commit message: Changed capacitor values and component layout
Parts:
- C13: renamed from C15; footprint Capacitors_SMD:C_0603 -> Capacitors_SMD:C_0805
- C14: renamed from C16; footprint Capacitors_SMD:C_0603 -> Capacitors_SMD:C_0805
- C15: renamed from C17; footprint Capacitors_SMD:C_0603 -> Capacitors_SMD:C_0805
- C16: renamed from C18; footprint Capacitors_SMD:C_0603 -> Capacitors_SMD:C_0805
- C25, C26, C27, C28, C29, C30, C31, C32: value 0.33uF -> 0.1uF; footprint Capacitors_SMD:C_0603 -> Capacitors_SMD:C_0402
Changed lines of the file:
@@
 P 3550 1300
 F 0 "C26" H 3665 1346 50  0000 L CNN
-F 1 "0.33uF" H 3665 1255 50  0000 L CNN
-F 2 "Capacitors_SMD:C_0603" H 3588 1150 50  0001 C CNN
+F 1 "0.1uF" H 3665 1255 50  0000 L CNN
+F 2 "Capacitors_SMD:C_0402" H 3588 1150 50  0001 C CNN
 F 3 "" H 3550 1300 50  0001 C CNN
 	1    3550 1300
@@
 P 2250 1300
 F 0 "C25" H 2365 1346 50  0000 L CNN
-F 1 "0.33uF" H 2365 1255 50  0000 L CNN
-F 2 "Capacitors_SMD:C_0603" H 2288 1150 50  0001 C CNN
+F 1 "0.1uF" H 2365 1255 50  0000 L CNN
+F 2 "Capacitors_SMD:C_0402" H 2288 1150 50  0001 C CNN
 F 3 "" H 2250 1300 50  0001 C CNN
 	1    2250 1300
@@
 	1650 2000 1850 2000
 $Comp
-L device:C C15
+L device:C C13
 U 1 1 5A957669
 P 1850 2400
-F 0 "C15" H 1965 2446 50  0000 L CNN
+F 0 "C13" H 1965 2446 50  0000 L CNN
 F 1 "0.1uF" H 1965 2355 50  0000 L CNN
-F 2 "Capacitors_SMD:C_0603" H 1888 2250 50  0001 C CNN
+F 2 "Capacitors_SMD:C_0805" H 1888 2250 50  0001 C CNN
 F 3 "" H 1850 2400 50  0001 C CNN
 	1    1850 2400
@@
 P 3600 4000
 F 0 "C30" H 3715 4046 50  0000 L CNN
-F 1 "0.33uF" H 3715 3955 50  0000 L CNN
-F 2 "Capacitors_SMD:C_0603" H 3638 3850 50  0001 C CNN
+F 1 "0.1uF" H 3715 3955 50  0000 L CNN
+F 2 "Capacitors_SMD:C_0402" H 3638 3850 50  0001 C CNN
 F 3 "" H 3600 4000 50  0001 C CNN
 	1    3600 4000
@@
 P 2300 4000
 F 0 "C29" H 2415 4046 50  0000 L CNN
-F 1 "0.33uF" H 2415 3955 50  0000 L CNN
-F 2 "Capacitors_SMD:C_0603" H 2338 3850 50  0001 C CNN
+F 1 "0.1uF" H 2415 3955 50  0000 L CNN
+F 2 "Capacitors_SMD:C_0402" H 2338 3850 50  0001 C CNN
 F 3 "" H 2300 4000 50  0001 C CNN
 	1    2300 4000
@@
 	1700 4700 1900 4700
 $Comp
-L device:C C17
+L device:C C15
 U 1 1 5A96C98B
 P 1900 5100
-F 0 "C17" H 2015 5146 50  0000 L CNN
+F 0 "C15" H 2015 5146 50  0000 L CNN
 F 1 "0.1uF" H 2015 5055 50  0000 L CNN
-F 2 "Capacitors_SMD:C_0603" H 1938 4950 50  0001 C CNN
+F 2 "Capacitors_SMD:C_0805" H 1938 4950 50  0001 C CNN
 F 3 "" H 1900 5100 50  0001 C CNN
 	1    1900 5100
@@
 P 7550 1300
 F 0 "C28" H 7665 1346 50  0000 L CNN
-F 1 "0.33uF" H 7665 1255 50  0000 L CNN
-F 2 "Capacitors_SMD:C_0603" H 7588 1150 50  0001 C CNN
+F 1 "0.1uF" H 7665 1255 50  0000 L CNN
+F 2 "Capacitors_SMD:C_0402" H 7588 1150 50  0001 C CNN
 F 3 "" H 7550 1300 50  0001 C CNN
 	1    7550 1300
@@
 P 6250 1300
 F 0 "C27" H 6365 1346 50  0000 L CNN
-F 1 "0.33uF" H 6365 1255 50  0000 L CNN
-F 2 "Capacitors_SMD:C_0603" H 6288 1150 50  0001 C CNN
+F 1 "0.1uF" H 6365 1255 50  0000 L CNN
+F 2 "Capacitors_SMD:C_0402" H 6288 1150 50  0001 C CNN
 F 3 "" H 6250 1300 50  0001 C CNN
 	1    6250 1300
@@
 	5650 2000 5850 2000
 $Comp
-L device:C C16
+L device:C C14
 U 1 1 5A96DD5B
 P 5850 2400
-F 0 "C16" H 5965 2446 50  0000 L CNN
+F 0 "C14" H 5965 2446 50  0000 L CNN
 F 1 "0.1uF" H 5965 2355 50  0000 L CNN
-F 2 "Capacitors_SMD:C_0603" H 5888 2250 50  0001 C CNN
+F 2 "Capacitors_SMD:C_0805" H 5888 2250 50  0001 C CNN
 F 3 "" H 5850 2400 50  0001 C CNN
 	1    5850 2400
@@
 P 7650 4000
 F 0 "C32" H 7765 4046 50  0000 L CNN
-F 1 "0.33uF" H 7765 3955 50  0000 L CNN
-F 2 "Capacitors_SMD:C_0603" H 7688 3850 50  0001 C CNN
+F 1 "0.1uF" H 7765 3955 50  0000 L CNN
+F 2 "Capacitors_SMD:C_0402" H 7688 3850 50  0001 C CNN
 F 3 "" H 7650 4000 50  0001 C CNN
 	1    7650 4000
@@
 P 6350 4000
 F 0 "C31" H 6465 4046 50  0000 L CNN
-F 1 "0.33uF" H 6465 3955 50  0000 L CNN
-F 2 "Capacitors_SMD:C_0603" H 6388 3850 50  0001 C CNN
+F 1 "0.1uF" H 6465 3955 50  0000 L CNN
+F 2 "Capacitors_SMD:C_0402" H 6388 3850 50  0001 C CNN
 F 3 "" H 6350 4000 50  0001 C CNN
 	1    6350 4000
@@
 	5750 4700 5950 4700
 $Comp
-L device:C C18
+L device:C C16
 U 1 1 5A970207
 P 5950 5100
-F 0 "C18" H 6065 5146 50  0000 L CNN
+F 0 "C16" H 6065 5146 50  0000 L CNN
 F 1 "0.1uF" H 6065 5055 50  0000 L CNN
-F 2 "Capacitors_SMD:C_0603" H 5988 4950 50  0001 C CNN
+F 2 "Capacitors_SMD:C_0805" H 5988 4950 50  0001 C CNN
 F 3 "" H 5950 5100 50  0001 C CNN
 	1    5950 5100

Commit message: Changed the microcontroller from qfn to tqfp
Parts:
- C10, C11, C13, C14, C15, C16, C25, C26, C27, C28, C29, C30, C31, C32, C4, C5, C6, C7, C8, C9: symbol device:C -> Thermocouple-Data-Logger-rescue:C-device
- J2, J3, J4, J5: symbol Connector:Conn_01x02 -> Thermocouple-Data-Logger-rescue:Conn_01x02-Connector
- R0, R1, R2, R3, R4, R5, R6, R7: symbol device:R -> Thermocouple-Data-Logger-rescue:R-device
- U2, U3, U4, U5: symbol sensors:MAX31856 -> Thermocouple-Data-Logger-rescue:MAX31856-sensors
Changed lines of the file:
@@
 $EndDescr
 $Comp
-L sensors:MAX31856 U2
+L Thermocouple-Data-Logger-rescue:MAX31856-sensors U2
 U 1 1 5A878CB3
 P 2900 2450
@@
 $EndComp
 $Comp
-L device:R R0
+L Thermocouple-Data-Logger-rescue:R-device R0
 U 1 1 5A8A855F
 P 1500 2000
@@
 $EndComp
 $Comp
-L device:R R1
+L Thermocouple-Data-Logger-rescue:R-device R1
 U 1 1 5A8A859A
 P 1500 2800
@@
 $EndComp
 $Comp
-L Connector:Conn_01x02 J2
+L Thermocouple-Data-Logger-rescue:Conn_01x02-Connector J2
 U 1 1 5A8A7D94
 P 1000 2450
@@
 VCC1
 $Comp
-L device:C C26
+L Thermocouple-Data-Logger-rescue:C-device C26
 U 1 1 5A8AA4BE
 P 3550 1300
@@
 $EndComp
 $Comp
-L device:C C25
+L Thermocouple-Data-Logger-rescue:C-device C25
 U 1 1 5A8AA592
 P 2250 1300
@@
 	1650 2000 1850 2000
 $Comp
-L device:C C13
+L Thermocouple-Data-Logger-rescue:C-device C13
 U 1 1 5A957669
 P 1850 2400
@@
 	1850 2800 2200 2800
 $Comp
-L device:C C5
+L Thermocouple-Data-Logger-rescue:C-device C5
 U 1 1 5A959D53
 P 1850 2950
@@
 	1850 3200 1850 3100
 $Comp
-L device:C C4
+L Thermocouple-Data-Logger-rescue:C-device C4
 U 1 1 5A95A909
 P 1850 1850
@@
 SDI
 $Comp
-L sensors:MAX31856 U4
+L Thermocouple-Data-Logger-rescue:MAX31856-sensors U4
 U 1 1 5A96C92D
 P 2950 5150
@@
 $EndComp
 $Comp
-L device:R R4
+L Thermocouple-Data-Logger-rescue:R-device R4
 U 1 1 5A96C942
 P 1550 4700
@@
 $EndComp
 $Comp
-L device:R R5
+L Thermocouple-Data-Logger-rescue:R-device R5
 U 1 1 5A96C949
 P 1550 5500
@@
 $EndComp
 $Comp
-L Connector:Conn_01x02 J4
+L Thermocouple-Data-Logger-rescue:Conn_01x02-Connector J4
 U 1 1 5A96C950
 P 1050 5150
@@
 VCC3
 $Comp
-L device:C C30
+L Thermocouple-Data-Logger-rescue:C-device C30
 U 1 1 5A96C962
 P 3600 4000
@@
 $EndComp
 $Comp
-L device:C C29
+L Thermocouple-Data-Logger-rescue:C-device C29
 U 1 1 5A96C969
 P 2300 4000
@@
 	1700 4700 1900 4700
 $Comp
-L device:C C15
+L Thermocouple-Data-Logger-rescue:C-device C15
 U 1 1 5A96C98B
 P 1900 5100
@@
 	1900 5500 2250 5500
 $Comp
-L device:C C9
+L Thermocouple-Data-Logger-rescue:C-device C9
 U 1 1 5A96C998
 P 1900 5650
@@
 	1900 5900 1900 5800
 $Comp
-L device:C C8
+L Thermocouple-Data-Logger-rescue:C-device C8
 U 1 1 5A96C9A6
 P 1900 4550
@@
 SDI
 $Comp
-L sensors:MAX31856 U3
+L Thermocouple-Data-Logger-rescue:MAX31856-sensors U3
 U 1 1 5A96DCFD
 P 6900 2450
@@
 $EndComp
 $Comp
-L device:R R2
+L Thermocouple-Data-Logger-rescue:R-device R2
 U 1 1 5A96DD12
 P 5500 2000
@@
 $EndComp
 $Comp
-L device:R R3
+L Thermocouple-Data-Logger-rescue:R-device R3
 U 1 1 5A96DD19
 P 5500 2800
@@
 $EndComp
 $Comp
-L Connector:Conn_01x02 J3
+L Thermocouple-Data-Logger-rescue:Conn_01x02-Connector J3
 U 1 1 5A96DD20
 P 5000 2450
@@
 VCC2
 $Comp
-L device:C C28
+L Thermocouple-Data-Logger-rescue:C-device C28
 U 1 1 5A96DD32
 P 7550 1300
@@
 $EndComp
 $Comp
-L device:C C27
+L Thermocouple-Data-Logger-rescue:C-device C27
 U 1 1 5A96DD39
 P 6250 1300
@@
 	5650 2000 5850 2000
 $Comp
-L device:C C14
+L Thermocouple-Data-Logger-rescue:C-device C14
 U 1 1 5A96DD5B
 P 5850 2400
@@
 	5850 2800 6200 2800
 $Comp
-L device:C C7
+L Thermocouple-Data-Logger-rescue:C-device C7
 U 1 1 5A96DD68
 P 5850 2950
@@
 	5850 3200 5850 3100
 $Comp
-L device:C C6
+L Thermocouple-Data-Logger-rescue:C-device C6
 U 1 1 5A96DD76
 P 5850 1850
@@
 SDI
 $Comp
-L sensors:MAX31856 U5
+L Thermocouple-Data-Logger-rescue:MAX31856-sensors U5
 U 1 1 5A9701A9
 P 7000 5150
@@
 $EndComp
 $Comp
-L device:R R6
+L Thermocouple-Data-Logger-rescue:R-device R6
 U 1 1 5A9701BE
 P 5600 4700
@@
 $EndComp
 $Comp
-L device:R R7
+L Thermocouple-Data-Logger-rescue:R-device R7
 U 1 1 5A9701C5
 P 5600 5500
@@
 $EndComp
 $Comp
-L Connector:Conn_01x02 J5
+L Thermocouple-Data-Logger-rescue:Conn_01x02-Connector J5
 U 1 1 5A9701CC
 P 5100 5150
@@
 VCC4
 $Comp
-L device:C C32
+L Thermocouple-Data-Logger-rescue:C-device C32
 U 1 1 5A9701DE
 P 7650 4000
@@
 $EndComp
 $Comp
-L device:C C31
+L Thermocouple-Data-Logger-rescue:C-device C31
 U 1 1 5A9701E5
 P 6350 4000
@@
 	5750 4700 5950 4700
 $Comp
-L device:C C16
+L Thermocouple-Data-Logger-rescue:C-device C16
 U 1 1 5A970207
 P 5950 5100
@@
 	5950 5500 6300 5500
 $Comp
-L device:C C11
+L Thermocouple-Data-Logger-rescue:C-device C11
 U 1 1 5A970214
 P 5950 5650
@@
 	5950 5900 5950 5800
 $Comp
-L device:C C10
+L Thermocouple-Data-Logger-rescue:C-device C10
 U 1 1 5A970222
 P 5950 4550
