File: Thermocouple-Data-Logger/Mounting_Hole.sch (KiCad schematic (older format))
At the start: 5 parts

Commit message: Finished general layout of large components
Parts:
- removed MK3, MK4: Mounting_Hole, Mounting_Holes:MountingHole_3.2mm_M3, symbol Mechanical:Mounting_Hole
- added MK2: Mounting_Hole_PAD, Mounting_Holes:MountingHole_3.2mm_M3_Pad_Via, symbol Mechanical:Mounting_Hole_PAD
- renumbered MK1 to MK0, MK2 to MK1, MK0 to MK3
Connections:
- wire segments 1 -> 2
Changed lines of the file:
@@
 $EndDescr
 $Comp
-L Mechanical:Mounting_Hole MK3
-U 1 1 5A9A8AAD
-P 3800 3250
-F 0 "MK3" H 3900 3296 50  0000 L CNN
-F 1 "Mounting_Hole" H 3900 3205 50  0000 L CNN
-F 2 "Mounting_Holes:MountingHole_3.2mm_M3" H 3800 3250 50  0001 C CNN
-F 3 "" H 3800 3250 50  0001 C CNN
-	1    3800 3250
-	1    0    0    -1
-$EndComp
-$Comp
-L Mechanical:Mounting_Hole_PAD MK0
+L Mechanical:Mounting_Hole_PAD MK3
 U 1 1 5A9A8B0C
-P 4850 2700
-F 0 "MK0" H 4950 2751 50  0000 L CNN
-F 1 "Mounting_Hole_PAD" H 4950 2660 50  0000 L CNN
-F 2 "Mounting_Holes:MountingHole_3.2mm_M3_Pad_Via" H 4850 2700 50  0001 C CNN
-F 3 "" H 4850 2700 50  0001 C CNN
-	1    4850 2700
+P 5800 3300
+F 0 "MK3" H 5900 3351 50  0000 L CNN
+F 1 "Mounting_Hole_PAD" H 5900 3260 50  0000 L CNN
+F 2 "Mounting_Holes:MountingHole_3.2mm_M3_Pad_Via" H 5800 3300 50  0001 C CNN
+F 3 "" H 5800 3300 50  0001 C CNN
+	1    5800 3300
 	1    0    0    -1
 $EndComp
@@
 L power:GND #PWR0184
 U 1 1 5A9A8BCE
-P 4850 2900
-F 0 "#PWR0184" H 4850 2650 50  0001 C CNN
-F 1 "GND" H 4855 2727 50  0000 C CNN
-F 2 "" H 4850 2900 50  0001 C CNN
-F 3 "" H 4850 2900 50  0001 C CNN
-	1    4850 2900
+P 5800 3500
+F 0 "#PWR0184" H 5800 3250 50  0001 C CNN
+F 1 "GND" H 5805 3327 50  0000 C CNN
+F 2 "" H 5800 3500 50  0001 C CNN
+F 3 "" H 5800 3500 50  0001 C CNN
+	1    5800 3500
 	1    0    0    -1
 $EndComp
 Wire Wire Line
-	4850 2900 4850 2800
+	5800 3500 5800 3400
 $Comp
-L Mechanical:Mounting_Hole MK4
-U 1 1 5A9A8DD7
-P 5850 3250
-F 0 "MK4" H 5950 3296 50  0000 L CNN
-F 1 "Mounting_Hole" H 5950 3205 50  0000 L CNN
-F 2 "Mounting_Holes:MountingHole_3.2mm_M3" H 5850 3250 50  0001 C CNN
-F 3 "" H 5850 3250 50  0001 C CNN
-	1    5850 3250
-	1    0    0    -1
-$EndComp
-$Comp
-L Mechanical:Mounting_Hole MK1
+L Mechanical:Mounting_Hole MK0
 U 1 1 5A9A8E2B
 P 3800 2000
-F 0 "MK1" H 3900 2046 50  0000 L CNN
+F 0 "MK0" H 3900 2046 50  0000 L CNN
 F 1 "Mounting_Hole" H 3900 1955 50  0000 L CNN
 F 2 "Mounting_Holes:MountingHole_3.2mm_M3" H 3800 2000 50  0001 C CNN
@@
 $EndComp
 $Comp
-L Mechanical:Mounting_Hole MK2
+L Mechanical:Mounting_Hole MK1
 U 1 1 5A9A8E5A
 P 5800 2000
-F 0 "MK2" H 5900 2046 50  0000 L CNN
+F 0 "MK1" H 5900 2046 50  0000 L CNN
 F 1 "Mounting_Hole" H 5900 1955 50  0000 L CNN
 F 2 "Mounting_Holes:MountingHole_3.2mm_M3" H 5800 2000 50  0001 C CNN
@@
 	1    0    0    -1
 $EndComp
+$Comp
+L Mechanical:Mounting_Hole_PAD MK2
+U 1 1 5A9D6481
+P 3800 3300
+F 0 "MK2" H 3900 3351 50  0000 L CNN
+F 1 "Mounting_Hole_PAD" H 3900 3260 50  0000 L CNN
+F 2 "Mounting_Holes:MountingHole_3.2mm_M3_Pad_Via" H 3800 3300 50  0001 C CNN
+F 3 "" H 3800 3300 50  0001 C CNN
+	1    3800 3300
+	1    0    0    -1
+$EndComp
+$Comp
+L power:GND #PWR?
+U 1 1 5A9D6488
+P 3800 3500
+F 0 "#PWR?" H 3800 3250 50  0001 C CNN
+F 1 "GND" H 3805 3327 50  0000 C CNN
+F 2 "" H 3800 3500 50  0001 C CNN
+F 3 "" H 3800 3500 50  0001 C CNN
+	1    3800 3500
+	1    0    0    -1
+$EndComp
+Wire Wire Line
+	3800 3500 3800 3400
 $EndSCHEMATC

Commit message: Satrted Labling the Components
Changed lines of the file:
@@
 Wire Wire Line
 	3800 3500 3800 3400
+$Comp
+L Graphic:Logo_Open_Hardware_Large #LOGO1
+U 1 1 5A9FD392
+P 4900 2700
+AR Path="/5A9A89AB/5A9FD392" Ref="#LOGO1"  Part="1"
+AR Path="/5A8E51AF/5A9FD392" Ref="#LOGO1"  Part="1"
+F 0 "#LOGO1" H 4900 3200 50  0001 C CNN
+F 1 "Logo_Open_Hardware_Large" H 4900 2300 50  0001 C CNN
+F 2 "Symbols:OSHW-Logo_11.4x12mm_SilkScreen" H 4900 2700 50  0001 C CNN
+F 3 "~" H 4900 2700 50  0001 C CNN
+	1    4900 2700
+	1    0    0    -1
+$EndComp
 $EndSCHEMATC
