File: Thermocouple-Data-Logger/Power.sch (KiCad schematic (older format))
At the start: 6 parts

Commit message: Added a lot more to the schimatic
Connections:
- net labels added: +5V
- wire segments 20 -> 21
Changed lines of the file:
@@
 Wire Wire Line
 	6750 2850 6750 3000
-Connection ~ 6750 2850
 Wire Wire Line
 	7950 2850 7950 2750
@@
 Wire Wire Line
 	4150 2850 4150 3050
-Connection ~ 5950 2850
 Wire Wire Line
 	5950 2850 5950 3050
@@
 	5450 2850 5950 2850
 Connection ~ 5450 2850
+Wire Wire Line
+	5450 2850 5450 2650
+$Comp
+L power:+5V #PWR?
+U 1 1 5A989E58
+P 5450 2650
+F 0 "#PWR?" H 5450 2500 50  0001 C CNN
+F 1 "+5V" H 5465 2823 50  0000 C CNN
+F 2 "" H 5450 2650 50  0001 C CNN
+F 3 "" H 5450 2650 50  0001 C CNN
+	1    5450 2650
+	1    0    0    -1
+$EndComp
 $EndSCHEMATC

Commit message: Added switches
Parts:
- gave numbers to parts that had none: 1
Changed lines of the file:
@@
 $EndComp
 $Comp
-L Thermocouple-Data-Logger:LT1763-3.3 U?
+L Thermocouple-Data-Logger:LT1763-3.3 U2
 U 1 1 5A8EC0FA
 P 6350 2950
-F 0 "U?" H 6350 3317 50  0000 C CNN
+F 0 "U2" H 6350 3317 50  0000 C CNN
 F 1 "LT1763-3.3" H 6350 3226 50  0000 C CNN
 F 2 "Housings_SOIC:SOIC-8_3.9x4.9mm_Pitch1.27mm" H 6350 3275 50  0001 C CNN

Commit message: Annotated schematic
Parts:
- J0: renamed from J?; value Conn_01x02 -> Power
- SW0: renamed from SW?; value SW_SPDT -> Power
- gave numbers to parts that had none: 3
- renumbered U2 to U1
Changed lines of the file:
@@
 $EndDescr
 $Comp
-L Switch:SW_SPDT SW?
+L Switch:SW_SPDT SW0
 U 1 1 5A8E52AA
 P 4650 2750
-F 0 "SW?" H 4650 3035 50  0000 C CNN
-F 1 "SW_SPDT" H 4650 2944 50  0000 C CNN
+F 0 "SW0" H 4650 3035 50  0000 C CNN
+F 1 "Power" H 4650 2944 50  0000 C CNN
 F 2 "" H 4650 2750 50  0001 C CNN
 F 3 "" H 4650 2750 50  0001 C CNN
@@
 $EndComp
 $Comp
-L device:C C?
+L device:C C40
 U 1 1 5A8E52B8
 P 5450 3000
-F 0 "C?" H 5565 3046 50  0000 L CNN
+F 0 "C40" H 5565 3046 50  0000 L CNN
 F 1 "10uF" H 5565 2955 50  0000 L CNN
 F 2 "" H 5488 2850 50  0001 C CNN
@@
 $EndComp
 $Comp
-L device:C C?
+L device:C C41
 U 1 1 5A8E52BF
 P 7600 3000
-F 0 "C?" H 7715 3046 50  0000 L CNN
+F 0 "C41" H 7715 3046 50  0000 L CNN
 F 1 "22uf" H 7715 2955 50  0000 L CNN
 F 2 "" H 7638 2850 50  0001 C CNN
@@
 $EndComp
 $Comp
-L device:C C?
+L device:C C12
 U 1 1 5A8E52C6
 P 7050 3000
-F 0 "C?" H 7165 3046 50  0000 L CNN
+F 0 "C12" H 7165 3046 50  0000 L CNN
 F 1 "0.01uF" H 7165 2955 50  0000 L CNN
 F 2 "" H 7088 2850 50  0001 C CNN
@@
 $EndComp
 $Comp
-L Connector:Conn_01x02 J?
+L Connector:Conn_01x02 J0
 U 1 1 5A8E52CE
 P 3750 2850
-F 0 "J?" H 3670 2525 50  0000 C CNN
-F 1 "Conn_01x02" H 3670 2616 50  0000 C CNN
+F 0 "J0" H 3670 2525 50  0000 C CNN
+F 1 "Power" H 3670 2616 50  0000 C CNN
 F 2 "" H 3750 2850 50  0001 C CNN
 F 3 "~" H 3750 2850 50  0001 C CNN
@@
 	3950 2750 4450 2750
 $Comp
-L power:GND #PWR?
+L power:GND #PWR0176
 U 1 1 5A8E52E6
 P 6350 3750
-F 0 "#PWR?" H 6350 3500 50  0001 C CNN
+F 0 "#PWR0176" H 6350 3500 50  0001 C CNN
 F 1 "GND" H 6355 3577 50  0000 C CNN
 F 2 "" H 6350 3750 50  0001 C CNN
@@
 $EndComp
 $Comp
-L power:+3.3V #PWR?
+L power:+3.3V #PWR0177
 U 1 1 5A8E52EF
 P 7950 2750
-F 0 "#PWR?" H 7950 2600 50  0001 C CNN
+F 0 "#PWR0177" H 7950 2600 50  0001 C CNN
 F 1 "+3.3V" H 7965 2923 50  0000 C CNN
 F 2 "" H 7950 2750 50  0001 C CNN
@@
 $EndComp
 $Comp
-L Thermocouple-Data-Logger:LT1763-3.3 U2
+L Thermocouple-Data-Logger:LT1763-3.3 U1
 U 1 1 5A8EC0FA
 P 6350 2950
-F 0 "U2" H 6350 3317 50  0000 C CNN
+F 0 "U1" H 6350 3317 50  0000 C CNN
 F 1 "LT1763-3.3" H 6350 3226 50  0000 C CNN
 F 2 "Housings_SOIC:SOIC-8_3.9x4.9mm_Pitch1.27mm" H 6350 3275 50  0001 C CNN
@@
 	4850 2850 5450 2850
 $Comp
-L power:GND #PWR?
+L power:GND #PWR0178
 U 1 1 5A8EC598
 P 5450 3300
-F 0 "#PWR?" H 5450 3050 50  0001 C CNN
+F 0 "#PWR0178" H 5450 3050 50  0001 C CNN
 F 1 "GND" H 5455 3127 50  0000 C CNN
 F 2 "" H 5450 3300 50  0001 C CNN
@@
 	6750 2850 7050 2850
 $Comp
-L power:GND #PWR?
+L power:GND #PWR0179
 U 1 1 5A8ED70D
 P 7600 3300
-F 0 "#PWR?" H 7600 3050 50  0001 C CNN
+F 0 "#PWR0179" H 7600 3050 50  0001 C CNN
 F 1 "GND" H 7605 3127 50  0000 C CNN
 F 2 "" H 7600 3300 50  0001 C CNN
@@
 	6750 3150 7050 3150
 $Comp
-L power:GND #PWR?
+L power:GND #PWR0180
 U 1 1 5A8EE196
 P 4150 3050
-F 0 "#PWR?" H 4150 2800 50  0001 C CNN
+F 0 "#PWR0180" H 4150 2800 50  0001 C CNN
 F 1 "GND" H 4155 2877 50  0000 C CNN
 F 2 "" H 4150 3050 50  0001 C CNN
@@
 	5450 2850 5450 2650
 $Comp
-L power:+5V #PWR?
+L power:+5V #PWR0181
 U 1 1 5A989E58
 P 5450 2650
-F 0 "#PWR?" H 5450 2500 50  0001 C CNN
+F 0 "#PWR0181" H 5450 2500 50  0001 C CNN
 F 1 "+5V" H 5465 2823 50  0000 C CNN
 F 2 "" H 5450 2650 50  0001 C CNN

Commit message: Made footprint for the terminal block
Parts:
- C12: footprint (none) -> Capacitors_SMD:C_0402
- C40: footprint (none) -> Capacitors_SMD:C_1210
- C41: footprint (none) -> Capacitors_SMD:C_1206
- J0: footprint (none) -> Connectors_JST:JST_PH_S2B-PH-SM4-TB_02x2.00mm_Angled
Changed lines of the file:
@@
 F 0 "C40" H 5565 3046 50  0000 L CNN
 F 1 "10uF" H 5565 2955 50  0000 L CNN
-F 2 "" H 5488 2850 50  0001 C CNN
+F 2 "Capacitors_SMD:C_1210" H 5488 2850 50  0001 C CNN
 F 3 "" H 5450 3000 50  0001 C CNN
 	1    5450 3000
@@
 F 0 "C41" H 7715 3046 50  0000 L CNN
 F 1 "22uf" H 7715 2955 50  0000 L CNN
-F 2 "" H 7638 2850 50  0001 C CNN
+F 2 "Capacitors_SMD:C_1206" H 7638 2850 50  0001 C CNN
 F 3 "" H 7600 3000 50  0001 C CNN
 	1    7600 3000
@@
 F 0 "C12" H 7165 3046 50  0000 L CNN
 F 1 "0.01uF" H 7165 2955 50  0000 L CNN
-F 2 "" H 7088 2850 50  0001 C CNN
+F 2 "Capacitors_SMD:C_0402" H 7088 2850 50  0001 C CNN
 F 3 "" H 7050 3000 50  0001 C CNN
 	1    7050 3000
@@
 F 0 "J0" H 3670 2525 50  0000 C CNN
 F 1 "Power" H 3670 2616 50  0000 C CNN
-F 2 "" H 3750 2850 50  0001 C CNN
+F 2 "Connectors_JST:JST_PH_S2B-PH-SM4-TB_02x2.00mm_Angled" H 3750 2850 50  0001 C CNN
 F 3 "~" H 3750 2850 50  0001 C CNN
 	1    3750 2850

Commit message: Added the components and generaterd the netlist
Parts:
- SW0: footprint (none) -> Buttons_Switches_SMD:SW_SPDT_CK-JS102011SAQN
Changed lines of the file:
@@
 F 0 "SW0" H 4650 3035 50  0000 C CNN
 F 1 "Power" H 4650 2944 50  0000 C CNN
-F 2 "" H 4650 2750 50  0001 C CNN
+F 2 "Buttons_Switches_SMD:SW_SPDT_CK-JS102011SAQN" H 4650 2750 50  0001 C CNN
 F 3 "" H 4650 2750 50  0001 C CNN
 	1    4650 2750
