File: Thermocouple-Data-Logger/Power.sch (KiCad schematic (older format))
At the start: 6 parts, among them J0 Power, SW0 Power, U1 LT1763-3.3

Commit message: Changed the microcontroller from qfn to tqfp
Parts:
- C12, C40, C41: symbol device:C -> Thermocouple-Data-Logger-rescue:C-device
- J0: symbol Connector:Conn_01x02 -> Thermocouple-Data-Logger-rescue:Conn_01x02-Connector
Changed lines of the file:
@@
 $EndComp
 $Comp
-L device:C C40
+L Thermocouple-Data-Logger-rescue:C-device C40
 U 1 1 5A8E52B8
 P 5450 3000
@@
 $EndComp
 $Comp
-L device:C C41
+L Thermocouple-Data-Logger-rescue:C-device C41
 U 1 1 5A8E52BF
 P 7600 3000
@@
 $EndComp
 $Comp
-L device:C C12
+L Thermocouple-Data-Logger-rescue:C-device C12
 U 1 1 5A8E52C6
 P 7050 3000
@@
 $EndComp
 $Comp
-L Connector:Conn_01x02 J0
+L Thermocouple-Data-Logger-rescue:Conn_01x02-Connector J0
 U 1 1 5A8E52CE
 P 3750 2850
