File: Thermocouple-Data-Logger/CLK2.sch (KiCad schematic (older format))
At the start: 3 parts

Commit message: Annotated schematic
Parts:
- gave numbers to parts that had none: 3
Changed lines of the file:
@@
 $EndDescr
 $Comp
-L device:Crystal Y?
+L device:Crystal Y1
 U 1 1 5A9FD744
 P 3600 3050
-F 0 "Y?" V 3554 3181 50  0000 L CNN
+F 0 "Y1" V 3554 3181 50  0000 L CNN
 F 1 "32.768KHz" V 3645 3181 50  0000 L CNN
 F 2 "" H 3600 3050 50  0001 C CNN
@@
 $EndComp
 $Comp
-L device:C C?
+L device:C C0
 U 1 1 5A9FD74B
 P 3900 2650
-F 0 "C?" V 4152 2650 50  0000 C CNN
+F 0 "C0" V 4152 2650 50  0000 C CNN
 F 1 "14pF" V 4061 2650 50  0000 C CNN
 F 2 "" H 3938 2500 50  0001 C CNN
@@
 $EndComp
 $Comp
-L device:C C?
+L device:C C1
 U 1 1 5A9FD752
 P 3900 3450
-F 0 "C?" V 3648 3450 50  0000 C CNN
+F 0 "C1" V 3648 3450 50  0000 C CNN
 F 1 "14pF" V 3739 3450 50  0000 C CNN
 F 2 "" H 3938 3300 50  0001 C CNN
@@
 	3600 3450 3750 3450
 $Comp
-L power:GND #PWR?
+L power:GND #PWR0182
 U 1 1 5A9FD75D
 P 4250 2650
-F 0 "#PWR?" H 4250 2400 50  0001 C CNN
+F 0 "#PWR0182" H 4250 2400 50  0001 C CNN
 F 1 "GND" H 4255 2477 50  0000 C CNN
 F 2 "" H 4250 2650 50  0001 C CNN
@@
 $EndComp
 $Comp
-L power:GND #PWR?
+L power:GND #PWR0183
 U 1 1 5A9FD763
 P 4250 3450
-F 0 "#PWR?" H 4250 3200 50  0001 C CNN
+F 0 "#PWR0183" H 4250 3200 50  0001 C CNN
 F 1 "GND" H 4255 3277 50  0000 C CNN
 F 2 "" H 4250 3450 50  0001 C CNN

Commit message: Made footprint for the terminal block
Parts:
- C0, C1: footprint (none) -> Capacitors_SMD:C_0402
Changed lines of the file:
@@
 F 0 "C0" V 4152 2650 50  0000 C CNN
 F 1 "14pF" V 4061 2650 50  0000 C CNN
-F 2 "" H 3938 2500 50  0001 C CNN
+F 2 "Capacitors_SMD:C_0402" H 3938 2500 50  0001 C CNN
 F 3 "" H 3900 2650 50  0001 C CNN
 	1    3900 2650
@@
 F 0 "C1" V 3648 3450 50  0000 C CNN
 F 1 "14pF" V 3739 3450 50  0000 C CNN
-F 2 "" H 3938 3300 50  0001 C CNN
+F 2 "Capacitors_SMD:C_0402" H 3938 3300 50  0001 C CNN
 F 3 "" H 3900 3450 50  0001 C CNN
 	1    3900 3450

Commit message: Added the components and generaterd the netlist
Parts:
- Y1: footprint (none) -> Crystals:Crystal_DS26_d2.0mm_l6.0mm_Horizontal
Changed lines of the file:
@@
 F 0 "Y1" V 3554 3181 50  0000 L CNN
 F 1 "32.768KHz" V 3645 3181 50  0000 L CNN
-F 2 "" H 3600 3050 50  0001 C CNN
+F 2 "Crystals:Crystal_DS26_d2.0mm_l6.0mm_Horizontal" H 3600 3050 50  0001 C CNN
 F 3 "" H 3600 3050 50  0001 C CNN
 	1    3600 3050

Commit message: Changed the microcontroller from qfn to tqfp
Parts:
- C0, C1: symbol device:C -> Thermocouple-Data-Logger-rescue:C-device
- Y1: symbol device:Crystal -> Thermocouple-Data-Logger-rescue:Crystal-device
Changed lines of the file:
@@
 $EndDescr
 $Comp
-L device:Crystal Y1
+L Thermocouple-Data-Logger-rescue:Crystal-device Y1
 U 1 1 5A9FD744
 P 3600 3050
@@
 $EndComp
 $Comp
-L device:C C0
+L Thermocouple-Data-Logger-rescue:C-device C0
 U 1 1 5A9FD74B
 P 3900 2650
@@
 $EndComp
 $Comp
-L device:C C1
+L Thermocouple-Data-Logger-rescue:C-device C1
 U 1 1 5A9FD752
 P 3900 3450
